File: v1.kicad_pcb (KiCad board)
At the start: 4 copper layers, 223.5 x 132.1 mm, 333 parts, among them J1 Powerpole G1377G2, J10 USB_B_Micro, J11 Micro_SD_Card_Det, J12 USB_A, J13 ARJM11D7-502-AB-EW2, J2 Barrel_Jack, J3 Conn_01x02, J4 Conn_01x02, J5 Conn_01x02, J6 Conn_01x02, J7 Conn_01x02, J8 Conn_01x02, J9 Conn_01x06_Male, M1 Logo_10mmx10mm, Q1 Si7141DP, Q10 SI1539CDL-T1-GE3, Q11 Si7141DP, Q12 SI1539CDL-T1-GE3, Q13 Si7141DP, Q14 SI1539CDL-T1-GE3, Q15 SI1539CDL-T1-GE3, Q2 SI1539CDL-T1-GE3, Q3 Si7141DP, Q4 SI1539CDL-T1-GE3, Q5 Si7141DP, Q6 Si7141DP, Q7 SI1539CDL-T1-GE3, Q8 SI1539CDL-T1-GE3, Q9 Si7141DP, SW1 SW_SPDT, SW2 SW_Push, T1 Transformer_SP_1S, U1 171050601, U10 NCP1117-3.3_TO252, U11 TLV803S, U12 MAX9612, U13 TPS3701DDCR, U14 MAX9612, U15 TPS3701DDCR, U16 LT3460, U17 MAX9612, U18 TPS3701DDCR, U19 LCMXO2-640HC-4SG48C, U2 MAX9612, U20 LTC2216, U21 TE0720, U22 JTAG-SMT3, U23 TPD2S017, U24 TXS02612, U25 TPS2051B, U26 TPD2S017, U27 AD5689RxCPZ, U3 TPS3701DDCR, U4 171050601, U5 MAX9612, U6 TPS3701DDCR, U7 NCP1117-3.3_TO252, U8 MAX9612, U9 TPS3701DDCR

Commit message: started layout
Parts:
- R125: value 7k5 -> 22k
- R127: value 22k -> 7k5
- moved C26 255.9 mm to (186.2, -191.1)
- moved D1 255.9 mm to (180.8, -196.6)
- moved R4 255.9 mm to (180.7, -156.8)
- moved R45 255.9 mm to (185.7, -197.5)
- moved R48 255.9 mm to (182.2, -191.1)
- moved BT1 255.9 mm to (22.5, -191.5)
- moved C1 255.9 mm to (184.9, -178.4)
- moved C10 255.9 mm to (145.1, -131.6)
- moved C11 255.9 mm to (139.5, -126.9)
- moved C12 255.9 mm to (136.3, -130.3)
- moved C13 255.9 mm to (80.5, -102.2)
- moved C14 255.9 mm to (80.5, -114.8)
- moved C15 255.9 mm to (80.5, -106.4)
- moved C16 255.9 mm to (54.2, -99.6)
- moved C17 255.9 mm to (74.9, -103.7)
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Connections:
- net Net-(U19-Pad18) renamed UART_PMIC_TO_FPGA
- net Net-(U19-Pad19) renamed UART_PMIC_FROM_FPGA
- J9 pad 2: Net-(J9-Pad2) -> /Power Supply/Power Rail Management/12V_VFault
- J9 pad 3: Net-(J9-Pad3) -> /Power Supply/Power Rail Management/12V_OK
- J9 pad 4: Net-(J9-Pad4) -> /Power Supply/Power Rail Management/12V_IFault
- J9 pad 5: Net-(J9-Pad5) -> /Power Supply/Power Rail Management/3V3_VFault
- LD10 pad 2: Net-(LD10-Pad2) -> GND
- LD10 pad 5: S3_PWR_ENABLE -> Net-(LD10-Pad5)
- LD2 pad 1: Net-(LD2-Pad1) -> GND
- LD2 pad 2: Net-(LD2-Pad2) -> GND
- LD2 pad 3: Net-(LD2-Pad3) -> GND
- LD2 pad 4: /Power Supply/Power Rail Management/12V_IFault -> Net-(LD2-Pad4)
- LD2 pad 5: /Power Supply/Power Rail Management/12V_OK -> Net-(LD2-Pad5)
- LD2 pad 6: /Power Supply/Power Rail Management/12V_VFault -> Net-(LD2-Pad6)
- LD3 pad 1: Net-(LD3-Pad1) -> GND
- LD3 pad 2: Net-(LD3-Pad2) -> GND
- LD3 pad 3: Net-(LD3-Pad3) -> GND
- LD3 pad 4: /Power Supply/Power Rail Management/3V3_IFault -> Net-(LD3-Pad4)
- LD3 pad 5: /Power Supply/Power Rail Management/3V3_OK -> Net-(LD3-Pad5)
- LD3 pad 6: /Power Supply/Power Rail Management/3V3_VFault -> Net-(LD3-Pad6)
- LD4 pad 1: Net-(LD4-Pad1) -> GND
- LD4 pad 2: Net-(LD4-Pad2) -> GND
- LD4 pad 3: Net-(LD4-Pad3) -> GND
- LD4 pad 4: /Power Supply/Power Rail Management/5V_IFault -> Net-(LD4-Pad4)
- LD4 pad 5: /Power Supply/Power Rail Management/5V_OK -> Net-(LD4-Pad5)
- LD4 pad 6: /Power Supply/Power Rail Management/5V_VFault -> Net-(LD4-Pad6)
- LD5 pad 1: Net-(LD5-Pad1) -> GND
- LD5 pad 2: Net-(LD5-Pad2) -> GND
- LD5 pad 3: Net-(LD5-Pad3) -> GND
- LD5 pad 4: /Power Supply/Power Rail Management/1V8_IFault -> Net-(LD5-Pad4)
- LD5 pad 5: /Power Supply/Power Rail Management/1V8_OK -> Net-(LD5-Pad5)
- LD5 pad 6: /Power Supply/Power Rail Management/1V8_VFault -> Net-(LD5-Pad6)
- LD6 pad 1: Net-(LD6-Pad1) -> GND
- LD6 pad 2: Net-(LD6-Pad2) -> GND
- LD6 pad 3: Net-(LD6-Pad3) -> GND
- LD6 pad 4: /Power Supply/Power Rail Management/3V3ADC_IFault -> Net-(LD6-Pad4)
- LD6 pad 5: /Power Supply/Power Rail Management/3V3ADC_OK -> Net-(LD6-Pad5)
- LD6 pad 6: /Power Supply/Power Rail Management/3V3ADC_VFault -> Net-(LD6-Pad6)
- LD7 pad 1: Net-(LD7-Pad1) -> GND
- LD7 pad 2: Net-(LD7-Pad2) -> GND
- LD7 pad 3: Net-(LD7-Pad3) -> GND
- LD7 pad 4: /Power Supply/Power Rail Management/16V_IFault -> Net-(LD7-Pad4)
- LD7 pad 5: 16V_OK -> Net-(LD7-Pad5)
- LD7 pad 6: /Power Supply/Power Rail Management/16V_VFault -> Net-(LD7-Pad6)
- LD8 pad 1: Net-(LD8-Pad1) -> GND
- LD8 pad 2: Net-(LD8-Pad2) -> GND
- LD8 pad 3: Net-(LD8-Pad3) -> GND
- LD8 pad 4: /Power Supply/Power Rail Management/UART_Error -> Net-(LD8-Pad4)
- LD8 pad 5: S1_PWR_ENABLE -> Net-(LD8-Pad5)
- LD8 pad 6: /Power Supply/Power Rail Management/I2C_Error -> Net-(LD8-Pad6)
- LD9 pad 2: Net-(LD9-Pad2) -> GND
- LD9 pad 5: S2_PWR_ENABLE -> Net-(LD9-Pad5)
- R107 pad 1: Net-(LD2-Pad1) -> /Power Supply/Power Rail Management/12V_VFault
- R107 pad 2: GND -> Net-(LD2-Pad6)
- R108 pad 1: Net-(LD2-Pad2) -> /Power Supply/Power Rail Management/12V_OK
- R108 pad 2: GND -> Net-(LD2-Pad5)
- R109 pad 1: Net-(LD2-Pad3) -> /Power Supply/Power Rail Management/12V_IFault
- R109 pad 2: GND -> Net-(LD2-Pad4)
- R110 pad 1: Net-(LD3-Pad1) -> /Power Supply/Power Rail Management/3V3_VFault
- R110 pad 2: GND -> Net-(LD3-Pad6)
- R111 pad 1: Net-(LD3-Pad2) -> /Power Supply/Power Rail Management/3V3_OK
- R111 pad 2: GND -> Net-(LD3-Pad5)
- R112 pad 1: Net-(LD3-Pad3) -> /Power Supply/Power Rail Management/3V3_IFault
- R112 pad 2: GND -> Net-(LD3-Pad4)
- R113 pad 1: Net-(LD4-Pad1) -> /Power Supply/Power Rail Management/5V_VFault
- R113 pad 2: GND -> Net-(LD4-Pad6)
- R114 pad 1: Net-(LD4-Pad2) -> /Power Supply/Power Rail Management/5V_OK
- R114 pad 2: GND -> Net-(LD4-Pad5)
- R115 pad 1: Net-(LD4-Pad3) -> /Power Supply/Power Rail Management/5V_IFault
- R115 pad 2: GND -> Net-(LD4-Pad4)
- R116 pad 1: Net-(LD5-Pad1) -> /Power Supply/Power Rail Management/1V8_VFault
- R116 pad 2: GND -> Net-(LD5-Pad6)
- R117 pad 1: Net-(LD5-Pad2) -> /Power Supply/Power Rail Management/1V8_OK
- R117 pad 2: GND -> Net-(LD5-Pad5)
- R118 pad 1: Net-(LD5-Pad3) -> /Power Supply/Power Rail Management/1V8_IFault
- R118 pad 2: GND -> Net-(LD5-Pad4)
- R119 pad 1: Net-(LD6-Pad1) -> /Power Supply/Power Rail Management/3V3ADC_VFault
- R119 pad 2: GND -> Net-(LD6-Pad6)
- R120 pad 1: Net-(LD6-Pad2) -> /Power Supply/Power Rail Management/3V3ADC_OK
- R120 pad 2: GND -> Net-(LD6-Pad5)
- R121 pad 1: Net-(LD6-Pad3) -> /Power Supply/Power Rail Management/3V3ADC_IFault
- R121 pad 2: GND -> Net-(LD6-Pad4)
- R122 pad 1: Net-(LD7-Pad1) -> /Power Supply/Power Rail Management/16V_VFault
- R122 pad 2: GND -> Net-(LD7-Pad6)
- R123 pad 1: Net-(LD7-Pad2) -> 16V_OK
- R123 pad 2: GND -> Net-(LD7-Pad5)
- R124 pad 1: Net-(LD7-Pad3) -> /Power Supply/Power Rail Management/16V_IFault
- R124 pad 2: GND -> Net-(LD7-Pad4)
- R125 pad 1: Net-(LD8-Pad1) -> /Power Supply/Power Rail Management/I2C_Error
- R125 pad 2: GND -> Net-(LD8-Pad4)
- R126 pad 1: Net-(LD8-Pad2) -> S1_PWR_ENABLE
- R126 pad 2: GND -> Net-(LD8-Pad5)
- R127 pad 1: Net-(LD8-Pad3) -> /Power Supply/Power Rail Management/UART_Error
- R127 pad 2: GND -> Net-(LD8-Pad6)
- R128 pad 1: Net-(LD9-Pad2) -> S2_PWR_ENABLE
- R128 pad 2: GND -> Net-(LD9-Pad5)
- R129 pad 1: Net-(LD10-Pad2) -> S3_PWR_ENABLE
- R129 pad 2: GND -> Net-(LD10-Pad5)
- U19 pad 10: Net-(U19-Pad10) -> /Power Supply/Power Rail Management/1V8_IFault
- U19 pad 11: Net-(U19-Pad11) -> /Power Supply/Power Rail Management/3V3ADC_VFault
- U19 pad 12: Net-(U19-Pad12) -> /Power Supply/Power Rail Management/3V3ADC_OK
- U19 pad 14: Net-(U19-Pad14) -> /Power Supply/Power Rail Management/3V3ADC_IFault
- U19 pad 15: Net-(U19-Pad15) -> /Power Supply/Power Rail Management/16V_VFault
- U19 pad 16: Net-(U19-Pad16) -> 16V_OK
- U19 pad 17: Net-(U19-Pad17) -> /Power Supply/Power Rail Management/16V_IFault
- U19 pad 2: Net-(U19-Pad2) -> /Power Supply/Power Rail Management/3V3_OK
- U19 pad 20: Net-(U19-Pad20) -> 12V_I_Good
- U19 pad 21: Net-(U19-Pad21) -> 12V_V_Good
- U19 pad 23: Net-(U19-Pad23) -> 3V3_I_Good
- U19 pad 24: Net-(U19-Pad24) -> 3V3_V_Good
- U19 pad 26: Net-(U19-Pad26) -> 5V_I_Good
- U19 pad 27: Net-(U19-Pad27) -> 5V_V_Good
- U19 pad 28: Net-(U19-Pad28) -> 1V8_I_Good
- U19 pad 29: Net-(U19-Pad29) -> 1V8_V_Good
- U19 pad 3: Net-(U19-Pad3) -> /Power Supply/Power Rail Management/3V3_IFault
- U19 pad 31: Net-(U19-Pad31) -> 3V3ADC_I_Good
- U19 pad 32: Net-(U19-Pad32) -> 3V3ADC_V_Good
- U19 pad 33: Net-(U19-Pad33) -> 16V_I_Good
- U19 pad 34: Net-(U19-Pad34) -> 16V_V_Good
- U19 pad 35: Net-(U19-Pad35) -> S3_PWR_ENABLE
- U19 pad 36: Net-(U19-Pad36) -> S2_PWR_ENABLE
- U19 pad 37: Net-(U19-Pad37) -> /Power Supply/Power Rail Management/UART_Error
- U19 pad 38: Net-(U19-Pad38) -> S1_PWR_ENABLE
- U19 pad 4: Net-(U19-Pad4) -> /Power Supply/Power Rail Management/5V_VFault
- U19 pad 40: Net-(U19-Pad40) -> /Power Supply/Power Rail Management/I2C_Error
- U19 pad 44: Net-(J9-Pad2) -> /Power Supply/Power Rail Management/12V_VFault
- U19 pad 45: Net-(J9-Pad3) -> /Power Supply/Power Rail Management/12V_OK
- U19 pad 47: Net-(J9-Pad4) -> /Power Supply/Power Rail Management/12V_IFault
- U19 pad 48: Net-(J9-Pad5) -> /Power Supply/Power Rail Management/3V3_VFault
- U19 pad 5: Net-(U19-Pad5) -> /Power Supply/Power Rail Management/5V_OK
- U19 pad 7: Net-(U19-Pad7) -> /Power Supply/Power Rail Management/5V_IFault
- U19 pad 8: Net-(U19-Pad8) -> /Power Supply/Power Rail Management/1V8_VFault
- U19 pad 9: Net-(U19-Pad9) -> /Power Supply/Power Rail Management/1V8_OK
- U20 pad 31: OGnd -> GND
- U20 pad 50: OGnd -> GND
- U21 pad 1.40: 1V8_FROM_FPGA -> 1V8_from_FPGA
Routing:
- net /Power Supply/Power Rail Management/16V_IFault: track 0.00 -> 33.6 mm
- net 16V_OK: track 0.00 -> 31.3 mm
- net /Power Supply/Power Rail Management/16V_VFault: track 0.00 -> 29.3 mm
- net /Power Supply/Power Rail Management/3V3ADC_IFault: track 0.00 -> 26.4 mm
- net /Power Supply/Power Rail Management/3V3ADC_OK: track 0.00 -> 25.2 mm
- net /Power Supply/Power Rail Management/3V3ADC_VFault: track 0.00 -> 23.9 mm
- net /Power Supply/Power Rail Management/1V8_IFault: track 0.00 -> 21.9 mm
- net /Power Supply/Power Rail Management/1V8_OK: track 0.00 -> 20.8 mm
- net /Power Supply/Power Rail Management/1V8_VFault: track 0.00 -> 19.8 mm
- net S3_PWR_ENABLE: track 0.00 -> 18.2 mm
- net /Power Supply/Power Rail Management/5V_IFault: track 0.00 -> 17.0 mm
- net /Power Supply/Power Rail Management/5V_OK: track 0.00 -> 16.5 mm
- net /Power Supply/Power Rail Management/5V_VFault: track 0.00 -> 15.4 mm
- net /Power Supply/Power Rail Management/12V_VFault: track 0.00 -> 13.6 mm
- net /Power Supply/Power Rail Management/12V_OK: track 0.00 -> 13.2 mm
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- added copper zone on F.Cu, net GND
Other:
- rule via_min_drill: 0.3 -> 0.2
- rule via_min_size: 0.4 -> 0.45
- board text added: "12V"
- board text added: "16V"
- board text added: "1V8"
- board text added: "3V3"
- board text added: "5V0"
- board text added: "ADC"
- board text added: "GND"
- board text added: "S1"
- board text added: "S2"
- board text added: "S3"
- board text added: "TCK"
- board text added: "TDI"
- board text added: "TDO"
- board text added: "TMS"

Commit message: started regulator layout
Parts:
- removed J2: Barrel_Jack, Connector_WUT:Barrel-Jack_Cliff_FC681478_TH
- F1: value 0ZCJ0035FF2G -> 150mA; footprint Diode_SMD:D_SOD-123 -> Resistor_SMD:R_1210_3225Metric
- J9: footprint Connector_JST:JST_PH_B6B-PH-K_1x06_P2.00mm_Vertical -> Connector_PinHeader_2.54mm:PinHeader_1x06_P2.54mm_Vertical_SMD_Pin1Left
- moved D3 318.8 mm to (144.0, 113.8), turned to 90 degrees
- moved R76 317.3 mm to (259.8, 130.5), turned to 270 degrees
- moved R75 317.2 mm to (248.5, 131.0), turned to 270 degrees
- moved R74 316.3 mm to (259.8, 127.2), turned to 270 degrees
- moved R15 312.7 mm to (214.5, 155.0), turned to 270 degrees
- moved R14 312.6 mm to (225.8, 151.2), turned to 270 degrees
- moved LD1 311.8 mm to (146.2, 108.6)
- moved R16 310.5 mm to (225.8, 154.5), turned to 270 degrees
- moved C27 309.7 mm to (138.2, 111.5), turned to 90 degrees
- moved D2 309.3 mm to (115.5, 102.8), turned to 270 degrees
- moved C28 309.2 mm to (131.5, 107.0)
- moved TP4 309.0 mm to (151.2, 115.4)
- moved R73 308.2 mm to (248.5, 127.2), turned to 270 degrees
- moved R70 307.6 mm to (263.2, 117.2), turned to 180 degrees
- moved R71 307.5 mm to (248.5, 123.5), turned to 270 degrees
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Connections:
- R1 pad 1: /Power Supply/Stage 2 Regulators/3V3_5A Regulator/Vout -> /Power Supply/Stage 2 Regulators/3V3 Monitor/Vin
- R1 pad 2: /Power Supply/Stage 2 Regulators/3V3 Monitor/Sense+ -> /Power Supply/Stage 2 Regulators/3V3 Monitor/Sense-
- R1 pad 3: /Power Supply/Stage 2 Regulators/3V3 Monitor/Sense- -> /Power Supply/Stage 2 Regulators/3V3 Monitor/Sense+
- R1 pad 4: /Power Supply/Stage 2 Regulators/3V3 Monitor/Vin -> /Power Supply/Stage 2 Regulators/3V3_5A Regulator/Vout
- R41 pad 1: Net-(C25-Pad1) -> /Power Supply/Stage 1 Regulators/12V Monitor/Vin
- R41 pad 2: /Power Supply/Stage 1 Regulators/12V Monitor/Sense+ -> /Power Supply/Stage 1 Regulators/12V Monitor/Sense-
- R41 pad 3: /Power Supply/Stage 1 Regulators/12V Monitor/Sense- -> /Power Supply/Stage 1 Regulators/12V Monitor/Sense+
- R41 pad 4: /Power Supply/Stage 1 Regulators/12V Monitor/Vin -> Net-(C25-Pad1)
- R58 pad 1: 1V8_from_FPGA -> /Power Supply/Stage 3 Regulators/1V8 Monitor/Vin
- R58 pad 2: /Power Supply/Stage 3 Regulators/1V8 Monitor/Sense+ -> /Power Supply/Stage 3 Regulators/1V8 Monitor/Sense-
- R58 pad 3: /Power Supply/Stage 3 Regulators/1V8 Monitor/Sense- -> /Power Supply/Stage 3 Regulators/1V8 Monitor/Sense+
- R58 pad 4: /Power Supply/Stage 3 Regulators/1V8 Monitor/Vin -> 1V8_from_FPGA
- R64 pad 1: Net-(C36-Pad1) -> /Power Supply/Stage 3 Regulators/ADC 3V3 Monitor/Vin
- R64 pad 2: /Power Supply/Stage 3 Regulators/ADC 3V3 Monitor/Sense+ -> /Power Supply/Stage 3 Regulators/ADC 3V3 Monitor/Sense-
- R64 pad 3: /Power Supply/Stage 3 Regulators/ADC 3V3 Monitor/Sense- -> /Power Supply/Stage 3 Regulators/ADC 3V3 Monitor/Sense+
- R64 pad 4: /Power Supply/Stage 3 Regulators/ADC 3V3 Monitor/Vin -> Net-(C36-Pad1)
- R9 pad 1: /Power Supply/Stage 2 Regulators/5V_5A Regulator/Vout -> /Power Supply/Stage 2 Regulators/5V Monitor/Vin
- R9 pad 2: /Power Supply/Stage 2 Regulators/5V Monitor/Sense+ -> /Power Supply/Stage 2 Regulators/5V Monitor/Sense-
- R9 pad 3: /Power Supply/Stage 2 Regulators/5V Monitor/Sense- -> /Power Supply/Stage 2 Regulators/5V Monitor/Sense+
- R9 pad 4: /Power Supply/Stage 2 Regulators/5V Monitor/Vin -> /Power Supply/Stage 2 Regulators/5V_5A Regulator/Vout
Routing:
- net GND: track 0.00 -> 150.0 mm, vias 0 -> 138
- net 3V3_LP: track 5.16 -> 83.6 mm
- net Net-(FL1-Pad3): track 0.00 -> 21.5 mm
- net /Power Supply/Stage 3 Regulators/16V Monitor/Sense-: track 0.00 -> 19.1 mm
- net Net-(J1-Pad1): track 0.00 -> 15.9 mm
- net /Power Supply/Stage 2 Regulators/12V_In: track 0.00 -> 13.0 mm, vias 0 -> 4
- net /Power Supply/Stage 3 Regulators/16V Step-up Regulator/16V_Out: track 0.00 -> 11.2 mm
- net /Power Supply/Stage 1 Regulators/Vin: track 0.00 -> 10.5 mm
- net Backlight_Vdd: track 0.00 -> 10.5 mm, vias 0 -> 4
- net +3V3: track 0.00 -> 10.5 mm, vias 0 -> 4
- net +3.3VADC: track 0.00 -> 10.5 mm, vias 0 -> 4
- net +1V8: track 0.00 -> 10.5 mm, vias 0 -> 4
- net +5V: track 0.00 -> 10.5 mm, vias 0 -> 4
- net /Power Supply/Stage 2 Regulators/5V Monitor/Sense-: track 0.00 -> 10.5 mm
- net /Power Supply/Stage 3 Regulators/ADC 3V3 Monitor/Sense-: track 0.00 -> 10.5 mm
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- added copper zone on F.Cu, net +1V8
- added copper zone on F.Cu, net +3.3VADC
- added copper zone on F.Cu, net +3V3
- added copper zone on F.Cu, net +5V
- added copper zone on F.Cu, net /Power Supply/Stage 1 Regulators/12V Monitor/Vin
- added copper zone on F.Cu, net /Power Supply/Stage 1 Regulators/Vin
- added copper zone on F.Cu, net /Power Supply/Stage 2 Regulators/12V_In
- added copper zone on F.Cu, net /Power Supply/Stage 2 Regulators/3V3 Monitor/Vin
- added copper zone on F.Cu, net /Power Supply/Stage 2 Regulators/5V Monitor/Vin
- added copper zone on F.Cu, net /Power Supply/Stage 3 Regulators/16V Monitor/Sense-
- added copper zone on F.Cu, net /Power Supply/Stage 3 Regulators/1V8 Monitor/Vin
- added copper zone on F.Cu, net /Power Supply/Stage 3 Regulators/ADC 3V3 Monitor/Vin
- added copper zone on F.Cu, net Backlight_Vdd
- added copper zone on In1.Cu, net GND
- added copper zone on F.Cu, net Net-(C25-Pad1)
Other:
- net class Default: clearance 0.0889 -> 0.1; via_dia 0.8 -> 0.45; via_drill 0.4 -> 0.2
- rule trace_clearance: 0.0889 -> 0.1
- board text added: "3V3_LP"
- board text added: "OFF"
- board text added: "ON"

Commit message: most of ADC front end done
Parts:
- added C100: 100n, Capacitor_SMD:C_0402_1005Metric, F.Cu at (91.8, 158.8)
- added C101: 100n, Capacitor_SMD:C_0402_1005Metric, F.Cu at (90.6, 149.7)
- added C102: 10u, Capacitor_SMD:C_0603_1608Metric, F.Cu at (71.8, 164.0)
- added C103: 100n, Capacitor_SMD:C_0603_1608Metric, F.Cu at (70.0, 164.0)
- added C104: 1n, Capacitor_SMD:C_0603_1608Metric, F.Cu at (68.2, 164.0)
- added C81: 10u, Capacitor_SMD:C_0603_1608Metric, F.Cu at (143.4, 99.4)
- added C82: 100n, Capacitor_SMD:C_0603_1608Metric, F.Cu at (162.4, 83.6)
- added C83: 1n, Capacitor_SMD:C_0603_1608Metric, F.Cu at (150.7, 89.6)
- added C84: 1u, Capacitor_SMD:C_0603_1608Metric, F.Cu at (160.1, 81.1)
- added C85: 10u, Capacitor_SMD:C_0603_1608Metric, F.Cu at (158.4, 84.2)
- added C86: 10u, Capacitor_SMD:C_0603_1608Metric, F.Cu at (147.7, 94.7)
- added C87: 100n, Capacitor_SMD:C_0603_1608Metric, F.Cu at (143.4, 96.9)
- added C88: 1n, Capacitor_SMD:C_0603_1608Metric, F.Cu at (164.5, 78.1)
- added C89: 100n, Capacitor_SMD:C_0402_1005Metric, F.Cu at (58.0, 137.0)
- added C90: 47p, Capacitor_SMD:C_0402_1005Metric, F.Cu at (60.4, 136.5)
- added C91: 150p, Capacitor_SMD:C_0402_1005Metric, F.Cu at (66.0, 136.5)
- added C92: 47p, Capacitor_SMD:C_0402_1005Metric, F.Cu at (71.6, 136.5)
- added C93: 22p, Capacitor_SMD:C_0402_1005Metric, F.Cu at (62.7, 156.9)
- added C94: 8p2, Capacitor_SMD:C_0402_1005Metric, F.Cu at (73.4, 156.9)
- added C95: 22p, Capacitor_SMD:C_0402_1005Metric, F.Cu at (80.3, 156.9)
- added C96: 100n, Capacitor_SMD:C_0402_1005Metric, F.Cu at (87.0, 156.9)
- added C97: 200p, Capacitor_SMD:C_0402_1005Metric, F.Cu at (67.3, 156.4)
- added C98: 200p, Capacitor_SMD:C_0402_1005Metric, F.Cu at (75.5, 156.4)
- added C99: 8p2, Capacitor_SMD:C_0402_1005Metric, F.Cu at (90.6, 147.8)
- added FB8: Ferrite_Bead_Small, Resistor_SMD:R_0603_1608Metric, F.Cu at (147.7, 92.1)
- added FB9: Ferrite_Bead_Small, Resistor_SMD:R_0603_1608Metric, F.Cu at (74.7, 164.8)
- added J14: Conn_Coaxial, Connector_WUT:SMA_Linx_CONSMA002-L-G_Horizontal, F.Cu at (52.4, 137.1)
- added J15: Conn_Coaxial, Connector_WUT:SMA_Linx_CONSMA002-L-G_Horizontal, F.Cu at (52.4, 156.9)
- added J2: Barrel_Jack, Connector_WUT:Barrel-Jack_Cliff_FC681478_TH, F.Cu at (39.9, -126.7)
- added L10: 24n, Inductor_SMD:L_0805_2012Metric, F.Cu at (77.7, 156.0)
- added L4: 330n, Inductor_SMD:L_0805_2012Metric, F.Cu at (63.2, 137.0)
- added L5: 330n, Inductor_SMD:L_0805_2012Metric, F.Cu at (68.8, 137.0)
- added L6: 220n, Inductor_SMD:L_0805_2012Metric, F.Cu at (59.5, 156.9)
- added L7: 560n, Inductor_SMD:L_0805_2012Metric, F.Cu at (70.0, 156.9)
- added L8: 220n, Inductor_SMD:L_0805_2012Metric, F.Cu at (83.7, 156.9)
- added L9: 24n, Inductor_SMD:L_0805_2012Metric, F.Cu at (65.3, 156.0)
- added R151: 10k, Resistor_SMD:R_0603_1608Metric, F.Cu at (164.1, 81.1)
- added R152: 51R, Resistor_SMD:R_0201_0603Metric, F.Cu at (89.6, 151.1)
- added R153: 0, Resistor_SMD:R_0603_1608Metric, F.Cu at (57.6, 164.2)
- added R154: 100R, Resistor_SMD:R_0402_1005Metric, F.Cu at (90.6, 143.8)
- added R155: 51R, Resistor_SMD:R_0201_0603Metric, F.Cu at (91.5, 151.1)
- added R156: 5R1, Resistor_SMD:R_0402_1005Metric, F.Cu at (90.1, 145.5)
- added R157: 5R1, Resistor_SMD:R_0402_1005Metric, F.Cu at (91.1, 145.5)
- added T2: Macom_ETC1-1-13, Transformer_SMD:Transformer_MACOM_SM-22, F.Cu at (90.6, 155.0)
- added TP8: TestPoint, TestPoint:TestPoint_Pad_D1.5mm, F.Cu at (158.5, 89.8)
- added U28: REF5025IDGK, Package_SO:MSOP-8_3x3mm_P0.65mm, F.Cu at (145.0, 87.4)
- added Y1: SIT5001AC-3E-33N0-80.000000X, Oscillator_WUT:TCXO_Sitime_SiT5001_5x3.2mm, F.Cu at (63.3, 163.9)
- T1: value Transformer_SP_1S -> PWB2010L; footprint Transformer_SMD:Transformer_MACOM_SM-22 -> Transformer_WUT:Coilcraft_PWB
- moved C10 432.8 mm to (-186.4, 99.5)
- moved C11 432.8 mm to (-179.7, 83.0)
- moved C12 432.8 mm to (-194.2, 87.5)
- moved C8 432.8 mm to (-171.2, 100.0)
- moved C9 432.8 mm to (-170.2, 97.5)
- moved J3 432.8 mm to (-175.7, 90.7)
- moved Q1 432.8 mm to (-188.4, 84.5)
- moved Q2 432.8 mm to (-180.9, 79.7)
- moved R1 432.8 mm to (-175.7, 85.5)
- moved R20 432.8 mm to (-188.4, 99.5)
- moved R21 432.8 mm to (-182.2, 83.0)
- moved R22 432.8 mm to (-183.4, 95.7)
- moved R23 432.8 mm to (-172.2, 97.5)
- moved R24 432.8 mm to (-173.7, 101.7)
- moved R25 432.8 mm to (-173.7, 103.5)
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Connections:
- R133 pad 2: Net-(R133-Pad2) -> Net-(C61-Pad2)
- R136 pad 2: Net-(R133-Pad2) -> Net-(C61-Pad2)
- R137 pad 1: Net-(R133-Pad2) -> Net-(C61-Pad2)
- T1 pad 1: Net-(R134-Pad2) -> Net-(C92-Pad1)
- T1 pad 2: Net-(R133-Pad2) -> (no net)
- T1 pad 3: Net-(R138-Pad2) -> GND
- T1 pad 4: Net-(T1-Pad4) -> Net-(R138-Pad2)
- T1 pad 5: Net-(T1-Pad5) -> Net-(C61-Pad2)
Routing:
- net GND: track 150.0 -> 194.2 mm, vias 138 -> 189
- net Net-(C61-Pad2): track 0.00 -> 20.3 mm
- net Net-(J15-Pad1): track 0.00 -> 13.1 mm
- net Net-(C59-Pad1): track 0.00 -> 9.80 mm
- net Net-(C102-Pad1): track 0.00 -> 9.44 mm
- net Net-(C99-Pad1): track 0.00 -> 7.63 mm
- net Net-(C99-Pad2): track 0.00 -> 7.60 mm
- net Net-(C62-Pad2): track 0.00 -> 6.78 mm
- net Net-(C60-Pad1): track 0.00 -> 6.77 mm
- net Net-(R154-Pad1): track 0.00 -> 6.31 mm
- net Net-(C94-Pad1): track 0.00 -> 5.94 mm
- net Net-(C93-Pad1): track 0.00 -> 5.91 mm
- net Net-(C92-Pad1): track 0.00 -> 5.23 mm
- net Net-(C89-Pad2): track 0.00 -> 5.12 mm
- net Net-(R154-Pad2): track 0.00 -> 5.01 mm
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Other:
- net class 50R_Microstrip added: clearance 0.2, trace_width 0.385, via_dia 0.45, via_drill 0.2
- board text added: "No coffee before soldering these ->"

Commit message: started laying out ADC
Parts:
- added C105: 100n, Capacitor_SMD:C_0402_1005Metric, F.Cu at (207.2, 60.5)
- added C106: 100n, Capacitor_SMD:C_0402_1005Metric, F.Cu at (228.0, 58.5)
- added C107: 100n, Capacitor_SMD:C_0402_1005Metric, F.Cu at (226.8, 58.5)
- added C108: 100n, Capacitor_SMD:C_0402_1005Metric, F.Cu at (229.3, 66.8)
- added C110: 1u, Capacitor_SMD:C_0603_1608Metric, F.Cu at (225.2, 56.8)
- added C111: 100n, Capacitor_SMD:C_0402_1005Metric, F.Cu at (211.3, 58.0)
- added C112: 100n, Capacitor_SMD:C_0402_1005Metric, F.Cu at (207.2, 62.5)
- added C113: 1u, Capacitor_SMD:C_0603_1608Metric, F.Cu at (206.2, 55.7)
- added FB10: Ferrite_Bead_Small, Resistor_SMD:R_0603_1608Metric, F.Cu at (223.5, 56.8)
- added FB11: Ferrite_Bead_Small, Resistor_SMD:R_0603_1608Metric, F.Cu at (195.5, 64.6)
- added LD13: LED_Cree_CLX6E-FKC, LED_SMD:LED_RGB_PLCC-6, F.Cu at (213.8, 78.5)
- added Q16: SI1539CDL-T1-GE3, Package_TO_SOT_SMD:SOT-363_SC-70-6, F.Cu at (218.0, 77.8)
- added R158: 0, Resistor_SMD:R_0603_1608Metric, F.Cu at (203.8, 59.6)
- added R159: 5k1, Resistor_SMD:R_0603_1608Metric, F.Cu at (220.5, 74.2)
- added R160: 10k, Resistor_SMD:R_0603_1608Metric, F.Cu at (220.5, 77.8)
- added R161: 10k, Resistor_SMD:R_0603_1608Metric, F.Cu at (223.0, 77.8)
- added R162: 22k, Resistor_SMD:R_0603_1608Metric, F.Cu at (218.0, 80.5)
- added U29: TLV7031DCK, Package_TO_SOT_SMD:SOT-353_SC-70-5, F.Cu at (218.0, 74.2)
- moved U22 365.2 mm to (240.8, 142.5), turned to 180 degrees
- moved J10 363.0 mm to (264.8, 142.5), turned to 90 degrees
- moved FL2 348.7 mm to (260.0, 142.5), turned to 180 degrees
- moved U21 348.0 mm to (185.5, 116.2), turned to 270 degrees
- moved U23 341.4 mm to (255.8, 142.5), turned to 90 degrees
- moved J13 339.2 mm to (260.8, 115.0), turned to 90 degrees
- moved J11 316.4 mm to (261.8, 95.5), turned to 270 degrees
- moved C78 312.4 mm to (243.7, 112.2), turned to 180 degrees
- moved U24 309.2 mm to (245.0, 96.8)
- moved J15 241.7 mm to (268.0, 47.6), turned to 270 degrees
- moved R153 239.8 mm to (262.9, 40.3), turned to 90 degrees
- moved Y1 229.8 mm to (257.2, 40.6), turned to 0 degrees
- moved L6 229.2 mm to (261.0, 47.6), turned to 180 degrees
- moved J14 226.6 mm to (268.0, 67.4), turned to 270 degrees
- moved C93 223.6 mm to (257.8, 47.6), turned to 0 degrees
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Connections:
- net Net-(U20-Pad20) renamed ADC_DITH
- net Net-(U20-Pad21) renamed ADC_D0-
- net Net-(U20-Pad22) renamed ADC_D0+
- net Net-(U20-Pad23) renamed ADC_D1-
- net Net-(U20-Pad24) renamed ADC_D1+
- net Net-(U20-Pad25) renamed ADC_D2-
- net Net-(U20-Pad26) renamed ADC_D2+
- net Net-(U20-Pad27) renamed ADC_D3-
- net Net-(U20-Pad28) renamed ADC_D3+
- net Net-(U20-Pad29) renamed ADC_D4-
- net Net-(U20-Pad30) renamed ADC_D4+
- net Net-(U20-Pad33) renamed ADC_D5-
- net Net-(U20-Pad34) renamed ADC_D5+
- net Net-(U20-Pad35) renamed ADC_D6-
- net Net-(U20-Pad36) renamed ADC_D6+
- net Net-(U20-Pad37) renamed ADC_D7-
- net Net-(U20-Pad38) renamed ADC_D7+
- net Net-(U20-Pad39) renamed ADC_CLK-
- net Net-(U20-Pad40) renamed ADC_CLK+
- net Net-(U20-Pad41) renamed ADC_D8-
- net Net-(U20-Pad42) renamed ADC_D8+
- net Net-(U20-Pad43) renamed ADC_D9-
- net Net-(U20-Pad44) renamed ADC_D9+
- net Net-(U20-Pad45) renamed ADC_D10-
- net Net-(U20-Pad46) renamed ADC_D10+
- net Net-(U20-Pad47) renamed ADC_D11-
- net Net-(U20-Pad48) renamed ADC_D11+
- net Net-(U20-Pad51) renamed ADC_D12-
- net Net-(U20-Pad52) renamed ADC_D12+
- net Net-(U20-Pad53) renamed ADC_D13-
- net Net-(U20-Pad54) renamed ADC_D13+
- net Net-(U20-Pad55) renamed ADC_D14-
- net Net-(U20-Pad56) renamed ADC_D14+
- net Net-(U20-Pad57) renamed ADC_D15-
- net Net-(U20-Pad58) renamed ADC_D15+
- J10 pad 2: Net-(FL2-Pad2) -> Net-(FL2-Pad1)
- J10 pad 3: Net-(FL2-Pad4) -> Net-(FL2-Pad3)
- U20 pad 61: Net-(U20-Pad61) -> +3.3VADC
- U20 pad 63: Net-(U20-Pad63) -> ADC_RAND
- U21 pad 1.11: ETH_MDI1_M -> ETH_MDI1_N
- U23 pad 3: Net-(FL2-Pad1) -> Net-(FL2-Pad2)
- U23 pad 4: Net-(FL2-Pad3) -> Net-(FL2-Pad4)
Routing:
- net GND: track 194.2 -> 273.7 mm, vias 189 -> 255
- net Net-(FL1-Pad3): track 21.5 -> 86.0 mm, vias 0 -> 3
- net Net-(J1-Pad1): track 15.9 -> 64.9 mm, vias 0 -> 2
- net Net-(FL1-Pad1): track 8.20 -> 32.9 mm, vias 0 -> 3
- net Net-(C86-Pad1): track 0.00 -> 13.3 mm
- net VDD: track 0.00 -> 11.9 mm, vias 0 -> 1
- net Net-(R159-Pad2): track 0.00 -> 10.2 mm
- net +3.3VADC: track 10.5 -> 20.2 mm, vias 4 -> 6
- net Net-(U20-Pad59): track 0.00 -> 9.50 mm
- net ADC_RAND: track 0.00 -> 8.87 mm
- net Net-(U20-Pad60): track 0.00 -> 8.66 mm
- net Net-(C81-Pad1): track 0.00 -> 7.89 mm
- net +3V3: track 10.5 -> 17.3 mm, vias 4 -> 9
- net Net-(FL2-Pad1): track 0.00 -> 4.70 mm
- net Net-(C85-Pad1): track 0.00 -> 4.25 mm
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Other:
- outline, holes or cut-outs redrawn
- net class Ethernet added: clearance 0.1, trace_width 0.25, via_dia 0.45, via_drill 0.2
- board text added: "<- No coffee before soldering these"
- board text removed: "No coffee before soldering these ->"
