File: v1.kicad_pcb (KiCad board)
At the start: 4 copper layers, 223.5 x 132.1 mm, 397 parts, among them J1 Powerpole G1377G2, J10 USB_B_Micro, J11 Micro_SD_Card_Det, J12 USB_A, J13 ARJM11D7-502-AB-EW2, J14 Conn_Coaxial, J15 Conn_Coaxial, J2 Barrel_Jack, J3 Conn_01x02, J4 Conn_01x02, J5 Conn_01x02, J6 Conn_01x02, J7 Conn_01x02, J8 Conn_01x02, J9 Conn_01x06_Male, M1 Logo_10mmx10mm, Q1 Si7141DP, Q10 SI1539CDL-T1-GE3, Q11 Si7141DP, Q12 SI1539CDL-T1-GE3, Q13 Si7141DP, Q14 SI1539CDL-T1-GE3, Q15 SI1539CDL-T1-GE3, Q16 SI1539CDL-T1-GE3, Q2 SI1539CDL-T1-GE3, Q3 Si7141DP, Q4 SI1539CDL-T1-GE3, Q5 Si7141DP, Q6 Si7141DP, Q7 SI1539CDL-T1-GE3, Q8 SI1539CDL-T1-GE3, Q9 Si7141DP, SW1 SW_SPDT, SW2 SW_Push, T1 PWB2010L, T2 Macom_ETC1-1-13, U1 171050601, U10 NCP1117-3.3_TO252, U11 TLV803S, U12 MAX9612, U13 TPS3701DDCR, U14 MAX9612, U15 TPS3701DDCR, U16 LT3460, U17 MAX9612, U18 TPS3701DDCR, U19 LCMXO2-640HC-4SG48C, U2 MAX9612, U20 LTC2216, U21 TE0720, U22 JTAG-SMT3, U23 TPD2S017, U24 TXS02612, U25 TPS2051B, U26 TPD2S017, U27 AD5689RxCPZ, U28 REF5025IDGK, U29 TLV7031DCK, U3 TPS3701DDCR, U4 171050601, U5 MAX9612, U6 TPS3701DDCR, U7 NCP1117-3.3_TO252, U8 MAX9612, U9 TPS3701DDCR, Y1 SIT5001AC-3E-33N0-80.000000X

Commit message: connected ADC to FPGA
Parts:
- removed C105: 100n, Capacitor_SMD:C_0402_1005Metric
- removed U29: TLV7031DCK, Package_TO_SOT_SMD:SOT-353_SC-70-5
- added D5: TPD1E1B04DPYR, Diode_WUT:X1SON, F.Cu at (165.0, 117.1)
- added RN2: 100, Resistor_SMD:R_Array_Convex_4x0402, F.Cu at (118.5, 120.5)
- added RN3: 100, Resistor_SMD:R_Array_Convex_8x0602, F.Cu at (118.5, 124.5)
- added RN4: 100, Resistor_SMD:R_Array_Convex_8x0602, F.Cu at (118.5, 129.5)
- RN1: footprint Resistor_SMD:R_Cat16-4 -> Resistor_SMD:R_Array_Concave_4x0402
- SW2: value SW_Push -> Tactile_Switch_Generic
- moved BT1 350.4 mm to (113.0, 147.0), turned to 270 degrees
- moved C65 322.3 mm to (120.2, 113.5), turned to 180 degrees
- moved C66 305.2 mm to (120.2, 117.0), turned to 180 degrees
- moved C113 276.1 mm to (-38.8, 183.0), turned to 180 degrees
- moved R161 243.5 mm to (-19.5, 99.2), turned to 90 degrees
- moved J15 241.0 mm to (52.2, 154.9), turned to 90 degrees
- moved R159 239.2 mm to (-17.0, 102.8), turned to 90 degrees
- moved SW2 239.1 mm to (169.0, 116.8), turned to 90 degrees
- moved R153 239.0 mm to (57.4, 162.2), turned to 270 degrees
- moved R160 238.5 mm to (-17.0, 99.2), turned to 90 degrees
- moved C68 233.9 mm to (166.8, 117.5), turned to 270 degrees
- moved Q16 233.5 mm to (-14.5, 99.2), turned to 90 degrees
- moved R162 233.0 mm to (-14.5, 96.5), turned to 180 degrees
- moved C67 232.8 mm to (164.2, 113.5)
- moved J9 230.6 mm to (-66.8, -54.0)
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Connections:
- net ADC_CLK+ renamed Net-(U20-Pad40)
- SW2 pad 2: GND -> ~PS_RESET
- SW2 pad 3: (no net) -> GND
- SW2 pad 4: (no net) -> GND
- U20 pad 21: ADC_D0- -> (no net)
- U20 pad 22: ADC_D0+ -> (no net)
- U20 pad 23: ADC_D1- -> (no net)
- U20 pad 24: ADC_D1+ -> (no net)
- U20 pad 25: ADC_D2- -> (no net)
- U20 pad 26: ADC_D2+ -> (no net)
- U20 pad 27: ADC_D3- -> (no net)
- U20 pad 28: ADC_D3+ -> (no net)
- U20 pad 29: ADC_D4- -> (no net)
- U20 pad 30: ADC_D4+ -> (no net)
- U20 pad 33: ADC_D5- -> (no net)
- U20 pad 34: ADC_D5+ -> (no net)
- U20 pad 35: ADC_D6- -> (no net)
- U20 pad 36: ADC_D6+ -> (no net)
- U20 pad 37: ADC_D7- -> (no net)
- U20 pad 38: ADC_D7+ -> (no net)
- U20 pad 39: ADC_CLK- -> (no net)
- U20 pad 41: ADC_D8- -> ADC_Clk
- U20 pad 42: ADC_D8+ -> ADC_D0
- U20 pad 43: ADC_D9- -> ADC_D1
- U20 pad 44: ADC_D9+ -> ADC_D2
- U20 pad 45: ADC_D10- -> ADC_D3
- U20 pad 46: ADC_D10+ -> ADC_D4
- U20 pad 47: ADC_D11- -> ADC_D5
- U20 pad 48: ADC_D11+ -> ADC_D6
- U20 pad 51: ADC_D12- -> ADC_D7
- U20 pad 52: ADC_D12+ -> ADC_D8
- U20 pad 53: ADC_D13- -> ADC_D9
- U20 pad 54: ADC_D13+ -> ADC_D10
- U20 pad 55: ADC_D14- -> ADC_D11
- U20 pad 56: ADC_D14+ -> ADC_D12
- U20 pad 57: ADC_D15- -> ADC_D13
- U20 pad 58: ADC_D15+ -> ADC_D14
- U20 pad 59: Net-(U20-Pad59) -> ADC_D15
- U20 pad 60: Net-(U20-Pad60) -> ADC_Overflow
Routing:
- net ETH_MDI2_N: track 0.00 -> 65.1 mm
- net ETH_MDI0_N: track 0.00 -> 65.0 mm
- net ETH_MDI3_N: track 0.60 -> 65.6 mm
- net ETH_MDI3_P: track 0.00 -> 65.0 mm
- net ETH_MDI1_N: track 0.00 -> 65.0 mm, vias 0 -> 2
- net ETH_MDI2_P: track 0.00 -> 65.0 mm
- net ETH_MDI1_P: track 0.00 -> 65.0 mm, vias 0 -> 2
- net ETH_MDI0_P: track 0.00 -> 65.0 mm
- net Net-(FL1-Pad3): track 86.0 -> 43.1 mm, vias 3 -> 0
- net GND: track 273.7 -> 314.6 mm, vias 255 -> 360
- net +3V3: track 17.3 -> 51.6 mm, vias 9 -> 23
- net Net-(J1-Pad1): track 64.9 -> 31.9 mm, vias 2 -> 0
- net ADC_Overflow: track 1.99 -> 31.4 mm
- net ADC_D15: track 0.00 -> 29.0 mm
- net ADC_DITH: track 0.00 -> 28.6 mm
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Other:
- board size 223.5 x 132.1 mm -> 206 x 145 mm
- board text added: "Apparently these are hard to get the right way round ->"
- board text added: "No coffee before soldering these ->"
- board text added: "PS Reset"
- board text removed: "<- No coffee before soldering these"

Commit message: more ADC faffing
Parts:
- removed C38: 22u, Capacitor_SMD:C_1210_3225Metric
- added C105: 22u, Capacitor_SMD:C_1210_3225Metric, F.Cu at (111.0, 100.8)
- added D6: TPD1E1B04DPYR, Diode_WUT:X1SON, F.Cu at (112.0, 144.0)
- moved C36 265.0 mm to (59.8, 98.5), turned to 180 degrees
- moved U10 252.8 mm to (62.0, 93.8), turned to 180 degrees
- moved C37 244.2 mm to (53.0, 93.8), turned to 180 degrees
- moved C35 243.4 mm to (69.5, 91.5)
- moved R68 236.6 mm to (75.3, 116.8), turned to 0 degrees
- moved R86 235.1 mm to (75.3, 114.8), turned to 0 degrees
- moved C47 233.5 mm to (75.3, 112.8), turned to 0 degrees
- moved R66 232.3 mm to (71.6, 116.8), turned to 0 degrees
- moved R94 231.9 mm to (79.3, 104.0), turned to 270 degrees
- moved R93 229.8 mm to (77.6, 104.0), turned to 270 degrees
- moved R91 229.2 mm to (79.3, 100.0), turned to 270 degrees
- moved U15 229.1 mm to (71.6, 112.8), turned to 0 degrees
- moved R65 227.9 mm to (67.8, 116.8), turned to 0 degrees
- moved R69 227.5 mm to (74.8, 105.5), turned to 0 degrees
- moved R90 227.0 mm to (77.6, 100.0), turned to 270 degrees
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Connections:
- U21 pad 1.10: VCCIO_B35 -> +1V8
- U21 pad 1.12: VCCIO_B35 -> +1V8
Routing:
- net GND: track 314.6 -> 555.3 mm, vias 360 -> 405
- net +3.3VADC: track 20.2 -> 33.6 mm
- net Net-(C36-Pad1): track 0.00 -> 12.7 mm
- net +1V8: track 10.5 -> 15.0 mm, vias 4 -> 6
- net /FPGA/JB1/NOSEQ: track 3.85 -> 0.00 mm, vias 2 -> 0
- net Net-(BT1-Pad1): track 22.1 -> 25.1 mm
- net +5V: track 10.5 -> 13.1 mm
- net SD_DAT3: track 0.00 -> 1.85 mm, vias 0 -> 1
- net SD_DAT1: track 0.00 -> 1.85 mm, vias 0 -> 1
- net SD_CMD: track 0.00 -> 1.80 mm, vias 0 -> 1
- net SD_CLK: track 0.00 -> 1.40 mm, vias 0 -> 1
- net VCCIO_B35: track 1.35 -> 0.00 mm, vias 1 -> 0
- net SD_DAT2: track 0.00 -> 1.35 mm, vias 0 -> 1
- net SD_DAT0: track 0.00 -> 1.35 mm, vias 0 -> 1
- net (no net): vias 8 -> 12
