File: v1.kicad_pcb (KiCad board)
At the start: 4 copper layers, 206 x 145 mm, 400 parts, among them J1 Powerpole G1377G2, J10 USB_B_Micro, J11 Micro_SD_Card_Det, J12 USB_A, J13 ARJM11D7-502-AB-EW2, J14 Conn_Coaxial, J15 Conn_Coaxial, J2 Barrel_Jack, J3 Conn_01x02, J4 Conn_01x02, J5 Conn_01x02, J6 Conn_01x02, J7 Conn_01x02, J8 Conn_01x02, J9 Conn_01x06_Male, M1 Logo_10mmx10mm, Q1 Si7141DP, Q10 SI1539CDL-T1-GE3, Q11 Si7141DP, Q12 SI1539CDL-T1-GE3, Q13 Si7141DP, Q14 SI1539CDL-T1-GE3, Q15 SI1539CDL-T1-GE3, Q16 SI1539CDL-T1-GE3, Q2 SI1539CDL-T1-GE3, Q3 Si7141DP, Q4 SI1539CDL-T1-GE3, Q5 Si7141DP, Q6 Si7141DP, Q7 SI1539CDL-T1-GE3, Q8 SI1539CDL-T1-GE3, Q9 Si7141DP, SW1 SW_SPDT, SW2 Tactile_Switch_Generic, T1 PWB2010L, T2 Macom_ETC1-1-13, U1 171050601, U10 NCP1117-3.3_TO252, U11 TLV803S, U12 MAX9612, U13 TPS3701DDCR, U14 MAX9612, U15 TPS3701DDCR, U16 LT3460, U17 MAX9612, U18 TPS3701DDCR, U19 LCMXO2-640HC-4SG48C, U2 MAX9612, U20 LTC2216, U21 TE0720, U22 JTAG-SMT3, U23 TPD2S017, U24 TXS02612, U25 TPS2051B, U26 TPD2S017, U27 AD5689RxCPZ, U28 REF5025IDGK, U3 TPS3701DDCR, U4 171050601, U5 MAX9612, U6 TPS3701DDCR, U7 NCP1117-3.3_TO252, U8 MAX9612, U9 TPS3701DDCR, Y1 SIT5001AC-3E-33N0-80.000000X

Commit message: Finished ADC layout
Parts:
- removed BT1: CR2032, Battery:BatteryHolder_Keystone_103_1x20mm
- removed C105: 22u, Capacitor_SMD:C_1210_3225Metric
- removed C108: 100n, Capacitor_SMD:C_0402_1005Metric
- removed C110: 1u, Capacitor_SMD:C_0603_1608Metric
- removed the C39 at (97.3, -142.9)
- removed the C44 at (-142.9, 52.6)
- removed the C50 at (71.9, -85.7)
- removed the C54 at (-81.7, 156.9)
- removed the C55 at (-80.7, 154.4)
- removed the C56 at (-96.9, 156.4)
- removed the C57 at (-90.2, 139.9)
- removed the C81 at (75.0, 125.0)
- removed the C86 at (92.8, 125.1)
- removed the C89 at (57.8, 135.0)
- removed the D4 at (59.8, -85.9)
- removed D6: TPD1E1B04DPYR, Diode_WUT:X1SON
- removed the FB10 at (96.8, 145.8)
- removed the J14 at (52.2, 135.1)
- removed the J8 at (-86.2, 147.7)
- removed the L3 at (61.2, -90.9)
- removed LD13: LED_Cree_CLX6E-FKC, LED_SMD:LED_RGB_PLCC-6
- removed the LD8 at (-48.1, -46.5)
- removed the Q13 at (-98.9, 141.4)
- removed Q14: SI1539CDL-T1-GE3, Package_TO_SOT_SMD:SOT-363_SC-70-6
- removed the Q8 at (115.2, -158.1)
- removed the R100 at (-93.9, 152.7)
- removed the R101 at (-82.7, 154.4)
- removed the R102 at (-84.2, 158.7)
- removed the R103 at (-84.2, 160.4)
- removed the R104 at (-88.2, 136.7)
- removed the R105 at (-88.2, 158.7)
- removed the R106 at (-88.2, 160.4)
- removed the R122 at (-79.6, -18.1)
- removed the R123 at (-79.6, -16.6)
- removed the R124 at (-79.6, -15.1)
- removed R159: 5k1, Resistor_SMD:R_0603_1608Metric
- removed the R70 at (-86.2, 142.7)
- removed the R71 at (-100.9, 148.9)
- removed the R72 at (113.3, -145.5)
- removed the R73 at (-100.9, 152.7)
- removed the R74 at (-89.7, 152.7)
- removed the R75 at (-100.9, 156.4)
- removed the R76 at (-89.7, 155.9)
- removed the R95 at (66.8, -89.4)
- removed the R96 at (63.9, -86.1)
- removed the R97 at (71.0, -93.2)
- removed the R98 at (-98.9, 156.4)
- removed the R99 at (-92.4, 139.9)
- removed the RN4 at (118.5, 129.5)
- removed the TP7 at (-104.7, 140.2)
- removed the U11 at (109.7, -154.1)
- removed the U16 at (66.9, -92.6)
- removed the U17 at (-86.2, 154.4)
- removed the U21 at (142.2, 125.0)
- added C42: 22u, Capacitor_SMD:C_1210_3225Metric, F.Cu at (95.9, 113.0)
- added C66: 100n, Capacitor_SMD:C_0402_1005Metric, F.Cu at (57.8, 135.0)
- added FB2: Ferrite_Bead_Small, Resistor_SMD:R_0603_1608Metric, F.Cu at (66.5, 125.0)
- added H1: Shield, Shield_WUT:Shield_Masach_MS585-10_58.2x49.4x4.7mm_SMD, F.Cu at (78.6, 142.8)
- added J11: Conn_01x02_Male, Connector_Molex:Molex_KK-254_AE-6410-02A_1x02_P2.54mm_Vertical, F.Cu at (114.5, 145.2)
- added J9: Conn_Coaxial, Connector_WUT:SMA_Linx_CONSMA002-L-G_Horizontal, B.Cu at (54.2, 135.0)
- added LD10: LED_Cree_CLX6E-FKC, LED_SMD:LED_RGB_PLCC-6, F.Cu at (83.5, 114.5)
- added R120: 5k1, Resistor_SMD:R_0603_1608Metric, F.Cu at (85.5, 121.0)
- added R130: 33, Resistor_SMD:R_0603_1608Metric, F.Cu at (103.5, 144.2)
- added RN1: 33, Resistor_SMD:R_Array_Convex_8x0602, F.Cu at (104.2, 135.5)
- C51: value 4u7 -> 100n; footprint Capacitor_SMD:C_0603_1608Metric -> Capacitor_SMD:C_0402_1005Metric
- C52: value 22u -> 1u
- C53: value 47n -> 10u
- C58: value 22u -> 10u; footprint Capacitor_SMD:C_1210_3225Metric -> Capacitor_SMD:C_0603_1608Metric
- J10: renamed from J15; moved to B.Cu
- RN2: value 100 -> 33; footprint Resistor_SMD:R_Array_Convex_4x0402 -> Resistor_SMD:R_Array_Convex_8x0602
- RN3: value 100 -> 33; footprint Resistor_SMD:R_Array_Convex_8x0602 -> Resistor_SMD:R_Array_Convex_4x0402
- U18: value TPS3701DDCR -> TE0720; footprint Package_TO_SOT_SMD:SOT-23-6 -> IC_WUT:Trenz_TE0720
- U21: renamed from U24; moved to B.Cu
- moved R62 250.8 mm to (107.9, 109.0), turned to 0 degrees
- moved R70 248.8 mm to (107.9, 107.2), turned to 0 degrees
- moved R60 248.1 mm to (104.2, 109.2), turned to 0 degrees
- moved C40 246.5 mm to (107.9, 105.2), turned to 0 degrees
- moved R59 245.2 mm to (100.4, 109.2), turned to 0 degrees
- moved U12 243.4 mm to (104.2, 105.2), turned to 0 degrees
- moved TP5 243.3 mm to (91.7, 113.0), turned to 90 degrees
- moved U18 240.7 mm to (142.2, 125.0), turned to 0 degrees
- moved R78 240.0 mm to (111.9, 96.5), turned to 270 degrees
- moved R72 239.9 mm to (104.2, 102.2), turned to 180 degrees
- moved R77 238.4 mm to (110.2, 96.5), turned to 270 degrees
- moved R63 237.8 mm to (107.4, 98.0), turned to 0 degrees
- moved Q8 237.2 mm to (92.9, 107.2), turned to 270 degrees
- moved R75 235.6 mm to (111.9, 92.5), turned to 270 degrees
- moved R61 235.0 mm to (104.2, 98.0), turned to 0 degrees
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- renumbered C79 to C100, C80 to C101, C40 to C38, C41 to C39, C42 to C40, C43 to C41, C45 to C43, C46 to C44, C47 to C45, C48 to C46, C49 to C47, C106 to C49, C107 to C50, C82 to C54, C83 to C55, C84 to C56, C85 to C57, C87 to C59, C111 to C60, C112 to C61, C113 to C62, C59 to C63, C88 to C64, C60 to C65, C61 to C67, C90 to C68, C91 to C69, C92 to C70, C62 to C71, C63 to C72, C64 to C73, C93 to C74, C94 to C75, C95 to C76, C96 to C77, C97 to C78, C98 to C79, C99 to C80, C100 to C81, C101 to C82, C102 to C83, C103 to C84, C104 to C85, C65 to C86, C66 to C87, C67 to C88, C68 to C89, C69 to C90, C70 to C91, C71 to C92, C72 to C93, C73 to C94, C74 to C95, C75 to C96, C76 to C97, C77 to C98, C78 to C99, D5 to D4, FB8 to FB1, FB6 to FB10, FB7 to FB11, FB11 to FB3, FB9 to FB4, FB1 to FB5, FB2 to FB6, FB3 to FB7, FB4 to FB8, FB5 to FB9, J10 to J12, J11 to J13, J13 to J14, J12 to J15, J9 to J8, L4 to L3, L5 to L4, L6 to L5, L7 to L6, L8 to L7, L9 to L8, L10 to L9, LD10 to LD8, Q11 to Q10, Q12 to Q11, Q16 to Q12, Q15 to Q13, Q9 to Q8, Q10 to Q9, R119 to R100, R120 to R101, R121 to R102, R125 to R103, R126 to R104, R127 to R105, R128 to R106, R129 to R107, R130 to R108, R131 to R109, R132 to R110, R151 to R111, R133 to R112, R134 to R113, R135 to R114, R136 to R115, R137 to R116, R158 to R117, R138 to R118, R139 to R119, R160 to R121, R161 to R122, R156 to R123, R152 to R124, R153 to R125, R154 to R126, R155 to R127, R157 to R128, R162 to R129, R140 to R131, R141 to R132, R142 to R133, R143 to R134, R144 to R135, R145 to R136, R146 to R137, R147 to R138, R148 to R139, R149 to R140, R150 to R141, R77 to R70, R78 to R71, R79 to R72, R80 to R73, R81 to R74, R82 to R75, R83 to R76, R84 to R77, R85 to R78, R86 to R79, R87 to R80, R88 to R81, R89 to R82, R90 to R83, R91 to R84, R92 to R85, R93 to R86, R94 to R87, R107 to R88, R108 to R89, R109 to R90, R110 to R91, R111 to R92, R112 to R93, R113 to R94, R114 to R95, R115 to R96, R116 to R97, R117 to R98, R118 to R99, RN1 to RN4, TP8 to TP7, U12 to U11, U13 to U12, U14 to U13, U15 to U14, U19 to U15, U28 to U16, U20 to U17, U22 to U19, U23 to U20, U25 to U22, U26 to U23, U27 to U24
Connections:
- C51 pad 1: +5V -> VDD
- C52 pad 1: /Power Supply/Stage 3 Regulators/16V Step-up Regulator/16V_Out -> VDD
- C54 pad 1: Net-(C81-Pad1) (its old number) -> Net-(C53-Pad1)
- C55 pad 1: Net-(C81-Pad1) (its old number) -> Net-(C53-Pad1)
- C58 pad 1: Backlight_Vdd -> Net-(C58-Pad1)
- C59 pad 1: Net-(C86-Pad1) -> Net-(C58-Pad1)
- C64 pad 1: Net-(C86-Pad1) -> Net-(C58-Pad1)
- FB1 pad 1: Net-(C81-Pad1) (its old number) -> Net-(C53-Pad1)
- FB4 pad 1: +3.3VADC -> VDD
- LD8 pad 5: Net-(LD10-Pad5) -> Net-(LD8-Pad5)
- R103 pad 2: Net-(LD8-Pad4) (its old number) -> Net-(LD7-Pad4)
- R104 pad 2: Net-(LD8-Pad5) -> Net-(LD7-Pad5)
- R105 pad 2: Net-(LD8-Pad6) (its old number) -> Net-(LD7-Pad6)
- R106 pad 2: Net-(LD9-Pad5) -> Net-(LD8-Pad5)
- R107 pad 2: Net-(LD10-Pad5) -> Net-(LD9-Pad5)
- R111 pad 1: Net-(C86-Pad1) -> Net-(C58-Pad1)
- R122 pad 1: ADC_RAND -> Net-(R122-Pad1)
- RN2 pad 1: ADC_RAND -> Net-(RN2-Pad1)
- RN2 pad 2: ADC_Overflow -> Net-(RN2-Pad2)
- RN2 pad 3: ADC_D15 -> Net-(RN2-Pad3)
- RN2 pad 4: ADC_D14 -> Net-(RN2-Pad4)
- RN3 pad 1: ADC_D13 -> Net-(RN3-Pad1)
- RN3 pad 2: ADC_D12 -> Net-(R122-Pad1)
- RN3 pad 3: ADC_D11 -> Net-(RN3-Pad3)
- RN3 pad 4: ADC_D10 -> Net-(RN3-Pad4)
- RN3 pad 5: ADC_D9 -> ADC_D15
- RN3 pad 6: ADC_D8 -> ADC_Overflow
- RN3 pad 7: ADC_D7 -> ADC_RAND
- RN3 pad 8: ADC_D6 -> Net-(RN3-Pad8)
- TP7 pad 1: Net-(C86-Pad1) -> Net-(C58-Pad1)
- U15 pad 33: 16V_I_Good -> FPGA_PWR_GOOD
- U15 pad 34: 16V_V_Good -> Net-(U15-Pad34)
- U16 pad 2: Net-(C81-Pad1) (its old number) -> Net-(C53-Pad1)
- U17 pad 1: Net-(C86-Pad1) -> Net-(C58-Pad1)
- U17 pad 41: ADC_Clk -> Net-(RN1-Pad8)
- U17 pad 42: ADC_D0 -> Net-(RN1-Pad7)
- U17 pad 43: ADC_D1 -> Net-(RN1-Pad6)
- U17 pad 44: ADC_D2 -> Net-(RN1-Pad5)
- U17 pad 45: ADC_D3 -> Net-(RN1-Pad4)
- U17 pad 46: ADC_D4 -> Net-(RN1-Pad3)
- U17 pad 47: ADC_D5 -> Net-(RN1-Pad2)
- U17 pad 48: ADC_D6 -> Net-(RN1-Pad1)
- U17 pad 51: ADC_D7 -> Net-(RN2-Pad8)
- U17 pad 52: ADC_D8 -> Net-(RN2-Pad7)
- U17 pad 53: ADC_D9 -> Net-(RN2-Pad6)
- U17 pad 54: ADC_D10 -> Net-(RN2-Pad5)
- U17 pad 55: ADC_D11 -> Net-(RN2-Pad4)
- U17 pad 56: ADC_D12 -> Net-(RN2-Pad3)
- U17 pad 57: ADC_D13 -> Net-(RN2-Pad2)
- U17 pad 58: ADC_D14 -> Net-(RN2-Pad1)
- U17 pad 59: ADC_D15 -> Net-(RN3-Pad4)
- U17 pad 60: ADC_Overflow -> Net-(RN3-Pad3)
- U17 pad 61: +3.3VADC -> GND
- U17 pad 63: ADC_RAND -> Net-(R122-Pad1)
Routing:
- net VDD: track 13.2 -> 63.9 mm, vias 1 -> 7
- net Net-(R130-Pad1): track 0.00 -> 28.5 mm, vias 0 -> 2
- net OVDD: track 6.11 -> 31.8 mm, vias 0 -> 3
- net GND: track 555.3 -> 576.4 mm, vias 405 -> 412
- net ADC_DITH: track 28.6 -> 8.99 mm
- net /Power Supply/Stage 3 Regulators/16V Monitor/Sense-: track 19.1 -> 0.00 mm
- net Net-(J11-Pad1): track 0.00 -> 18.9 mm
- net Net-(LD10-Pad3): track 2.55 -> 19.9 mm, vias 0 -> 2
- net Net-(BT1-Pad1): track 25.1 -> 8.43 mm
- net Net-(R122-Pad1): track 0.00 -> 16.0 mm
- net Net-(R120-Pad2): track 4.03 -> 19.9 mm, vias 0 -> 2
- net Net-(RN3-Pad3): track 0.00 -> 13.6 mm
- net Net-(C86-Pad1): track 13.3 -> 0.00 mm
- net Net-(C58-Pad1): track 0.00 -> 13.3 mm
- net Net-(RN3-Pad4): track 0.00 -> 13.3 mm
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- added copper zone on In2.Cu, net +3.3VADC
- added copper zone on B.Cu, net GND
- added copper zone on In2.Cu, net VDD
- removed copper zone on F.Cu, net /Power Supply/Stage 3 Regulators/16V Monitor/Sense-
- removed copper zone on F.Cu, net Backlight_Vdd
Other:
- board text added: "(This is where the magic happens)"
- board text added: "+"
- board text added: "3V3 ADC"
- board text added: "3V3 LP"
- board text added: "ADC OF"
- board text added: "Battery"
- board text added: "Or you could just use a PICAXE..."

Commit message: bit more faffing
Parts:
- added H2: Shield, Shield_WUT:Shield_Masach_MS570-10_52.7x30.7x6mm_TH, F.Cu at (216.8, 97.8)
- added H3: Shield, Shield_WUT:Shield_Masach_MS570-10_52.7x30.7x6mm_TH, F.Cu at (206.8, 64.5)
- moved LD12 367.4 mm to (162.2, 165.8), turned to 180 degrees
- moved FL3 347.2 mm to (175.0, 154.2), turned to 270 degrees
- moved J15 346.0 mm to (175.0, 165.8)
- moved C100 344.5 mm to (168.8, 158.5), turned to 270 degrees
- moved R140 344.5 mm to (132.2, 165.5), turned to 90 degrees
- moved R137 343.3 mm to (171.5, 156.2), turned to 270 degrees
- moved U22 341.2 mm to (157.0, 157.0), turned to 180 degrees
- moved U23 339.4 mm to (175.0, 158.0), turned to 180 degrees
- moved C101 338.7 mm to (165.0, 158.5), turned to 270 degrees
- moved R141 338.2 mm to (130.0, 165.5), turned to 90 degrees
- moved R139 335.7 mm to (157.8, 164.5)
- moved R138 333.5 mm to (157.8, 167.0)
- moved C91 329.7 mm to (-68.0, 95.7)
- moved C92 329.7 mm to (-49.6, 72.1)
- moved C93 329.7 mm to (-61.5, 84.4)
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Connections:
- net Net-(J15-Pad2) renamed /FPGA/Connectors/D-
- net Net-(J15-Pad3) renamed /FPGA/Connectors/D+
- C16 pad 2: GND -> /Power Supply/Stage 2 Regulators/5V_5A Regulator/FB_Gnd
- C4 pad 2: GND -> /Power Supply/Stage 2 Regulators/3V3_5A Regulator/FB_Gnd
- R18 pad 2: GND -> /Power Supply/Stage 2 Regulators/3V3_5A Regulator/FB_Gnd
- R19 pad 2: GND -> /Power Supply/Stage 2 Regulators/3V3_5A Regulator/FB_Gnd
- R30 pad 2: GND -> /Power Supply/Stage 2 Regulators/5V_5A Regulator/FB_Gnd
- R31 pad 2: GND -> /Power Supply/Stage 2 Regulators/5V_5A Regulator/FB_Gnd
- U18 pad 1.97: Net-(U18-Pad1.97) -> ~ETH_Link
- U18 pad 1.99: Net-(U18-Pad1.99) -> ~ETH_Active
Routing:
- net GND: track 576.4 -> 919.7 mm, vias 412 -> 612
- net /Power Supply/Stage 2 Regulators/5V_5A Regulator/Vout: track 0.00 -> 79.1 mm
- net USB_OTG_D+: track 0.00 -> 72.9 mm
- net USB_OTG_D-: track 0.00 -> 72.7 mm, vias 0 -> 2
- net USB_OTG_VBUS: track 0.00 -> 68.3 mm, vias 0 -> 2
- net USB_OTG_VEN: track 0.00 -> 55.4 mm, vias 0 -> 2
- net /Power Supply/Stage 2 Regulators/5V_5A Regulator/FB_Gnd: track 0.00 -> 48.0 mm
- net Net-(R31-Pad1): track 0.00 -> 38.3 mm, vias 0 -> 10
- net Net-(C16-Pad1): track 0.00 -> 35.3 mm, vias 0 -> 10
- net /Power Supply/Power Rail Management/16V_IFault: track 33.6 -> 0.00 mm
- net /Power Supply/Stage 2 Regulators/3V3_5A Regulator/Vout: track 0.00 -> 31.6 mm
- net 16V_OK: track 31.3 -> 0.00 mm
- net ~ETH_Link: track 0.00 -> 31.1 mm
- net /Power Supply/Stage 2 Regulators/12V_In: track 13.0 -> 43.8 mm
- net Net-(R29-Pad2): track 0.00 -> 30.4 mm
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- added copper zone on F.Cu, net /Power Supply/Stage 2 Regulators/3V3_5A Regulator/Vout
- added copper zone on F.Cu, net /Power Supply/Stage 2 Regulators/5V_5A Regulator/Vout
- added copper zone on F.Cu, net Net-(C14-Pad1)
- added copper zone on F.Cu, net Net-(C2-Pad1)
Other:
- board text added: "ADC OVF"
- board text added: "USB OC"
- board text removed: "16V"
- board text removed: "ADC OF"
- board text removed: "Apparently these are hard to get the right way round ->"

Commit message: more stuff done
Parts:
- removed J11: Conn_01x02_Male, Connector_Molex:Molex_KK-254_AE-6410-02A_1x02_P2.54mm_Vertical
- removed R74, R75, R77, R78: R, Resistor_SMD:R_0603_1608Metric
- removed R76: 10k, Resistor_SMD:R_0603_1608Metric
- added C102: 10u, Capacitor_SMD:C_0603_1608Metric, F.Cu at (76.8, 48.5)
- added C103: 100n, Capacitor_SMD:C_0603_1608Metric, F.Cu at (78.5, 48.5)
- added C104: 100n, Capacitor_SMD:C_0603_1608Metric, F.Cu at (99.5, 47.0)
- added C105: 100n, Capacitor_SMD:C_0603_1608Metric, F.Cu at (96.2, 56.2)
- added C106: 10u, Capacitor_SMD:C_0603_1608Metric, F.Cu at (98.2, 41.2)
- added C107: 100n, Capacitor_SMD:C_0603_1608Metric, F.Cu at (94.8, 43.0)
- added C108: 10u, Capacitor_SMD:C_0603_1608Metric, F.Cu at (79.0, 44.0)
- added C109: 100n, Capacitor_SMD:C_0603_1608Metric, F.Cu at (80.8, 44.0)
- added C110: 100n, Capacitor_SMD:C_0603_1608Metric, F.Cu at (99.5, 48.8)
- added C111: 100n, Capacitor_SMD:C_0603_1608Metric, F.Cu at (62.8, 73.8)
- added FB12: BLM18RK601SN1D, Resistor_SMD:R_0603_1608Metric, F.Cu at (75.0, 48.5)
- added FB13: BLM18RK601SN1D, Resistor_SMD:R_0603_1608Metric, F.Cu at (98.2, 43.0)
- added FB14: BLM18RK601SN1D, Resistor_SMD:R_0603_1608Metric, F.Cu at (77.2, 44.0)
- added J17: HDMI_A, Connector_WUT:HDMI_Wurth_685119134923_Horizontal, F.Cu at (89.5, 31.0)
- added L10: 100uH, Inductor_WUT:Wurth_7447709101, F.Cu at (166.8, 154.2)
- added LD13: LED_Cree_CLX6E-FKC, LED_SMD:LED_RGB_PLCC-6, F.Cu at (103.2, 36.2)
- added R142: 0, Resistor_SMD:R_0603_1608Metric, F.Cu at (176.5, 56.5)
- added RN5: 33, Resistor_SMD:R_Cat16-8, F.Cu at (100.8, 58.2)
- added RN6: 33, Resistor_SMD:R_Cat16-8, F.Cu at (100.8, 67.0)
- C39: value 100n -> 4u7
- C41: value 4u7 -> 22u; footprint Capacitor_SMD:C_0603_1608Metric -> Capacitor_SMD:C_1210_3225Metric
- C42: value 22u -> 100nF; footprint Capacitor_SMD:C_1210_3225Metric -> Capacitor_SMD:C_0603_1608Metric
- R59: value 130k -> 10k
- R60: value 2k2 -> 47k
- R62: value 36k -> 27k
- R70: value 100R -> 10k
- R71: value 10k -> 510
- R72: value 47k -> 33k
- R73: value 47k -> 22k
- U12: value TPS3701DDCR -> TFP410PAP; footprint Package_TO_SOT_SMD:SOT-23-6 -> IC_WUT:TQFP-64-1EP_10x10mm_P0.5mm_EP5x5mm_ThermalVias
- U21: moved to F.Cu
- moved LD6 426.2 mm to (382.5, 17.2), turned to 180 degrees
- moved LD5 425.5 mm to (382.5, 23.2), turned to 180 degrees
- moved LD2 425.3 mm to (382.5, 41.2), turned to 180 degrees
- moved LD4 425.1 mm to (382.5, 29.2), turned to 180 degrees
- moved LD3 425.0 mm to (382.5, 35.2), turned to 180 degrees
- moved R102 414.5 mm to (376.5, 15.8), turned to 0 degrees
- moved R101 414.2 mm to (376.5, 17.2), turned to 0 degrees
- moved R100 414.0 mm to (376.5, 18.8), turned to 0 degrees
- moved R99 413.6 mm to (376.5, 21.8), turned to 0 degrees
- moved R98 413.5 mm to (376.5, 23.2), turned to 0 degrees
- moved R97 413.3 mm to (376.5, 24.8), turned to 0 degrees
- moved R96 413.1 mm to (376.5, 27.8), turned to 0 degrees
- moved R95 413.1 mm to (376.5, 29.2), turned to 0 degrees
- moved R91 413.1 mm to (376.5, 36.8), turned to 0 degrees
- moved R94 413.0 mm to (376.5, 30.8), turned to 0 degrees
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Connections:
- net /Power Supply/Stage 3 Regulators/1V8 Monitor/Sense+ renamed Net-(J6-Pad1)
- net /Power Supply/Stage 3 Regulators/1V8 Monitor/Sense- renamed Net-(J6-Pad2)
- net /Power Supply/Stage 3 Regulators/1V8 Monitor/SetV renamed Net-(R61-Pad2)
- net Net-(U18-Pad1.100) renamed UART_USER_FROM_FPGA
- net Net-(U18-Pad1.98) renamed UART_USER_TO_FPGA
- C1 pad 2: GND -> DGND
- C10 pad 2: GND -> DGND
- C100 pad 2: GND -> DGND
- C101 pad 2: GND -> DGND
- C11 pad 2: GND -> DGND
- C12 pad 2: GND -> DGND
- C13 pad 2: GND -> DGND
- C14 pad 2: GND -> DGND
- C15 pad 2: GND -> DGND
- C17 pad 2: GND -> DGND
- C18 pad 2: GND -> DGND
- C19 pad 2: GND -> DGND
- C2 pad 2: GND -> DGND
- C20 pad 2: GND -> DGND
- C21 pad 2: GND -> DGND
- C22 pad 2: GND -> DGND
- C23 pad 2: GND -> DGND
- C24 pad 2: GND -> DGND
- C25 pad 2: GND -> DGND
- C26 pad 2: GND -> DGND
- C27 pad 2: GND -> DGND
- C28 pad 2: GND -> DGND
- C29 pad 2: GND -> DGND
- C3 pad 2: GND -> DGND
- C30 pad 2: GND -> DGND
- C31 pad 2: GND -> DGND
- C32 pad 2: GND -> DGND
- C33 pad 2: GND -> DGND
- C34 pad 2: GND -> DGND
- C35 pad 2: GND -> DGND
- C36 pad 2: GND -> DGND
- C37 pad 2: GND -> DGND
- C38 pad 1: 3V3_LP -> Net-(C38-Pad1)
- C38 pad 2: GND -> DGND
- C39 pad 2: GND -> DGND
- C40 pad 1: Net-(C40-Pad1) -> 3V3_LP
- C40 pad 2: GND -> DGND
- C41 pad 1: /Power Supply/Stage 3 Regulators/1V8 Monitor/Vin -> +1V8
- C41 pad 2: GND -> DGND
- C42 pad 1: +1V8 -> Net-(C42-Pad1)
- C42 pad 2: GND -> DGND
- C43 pad 2: GND -> DGND
- C44 pad 2: GND -> DGND
- C45 pad 2: GND -> DGND
- C46 pad 2: GND -> DGND
- C47 pad 2: GND -> DGND
- C49 pad 2: GND -> DGND
- C5 pad 2: GND -> DGND
- C50 pad 2: GND -> DGND
- C51 pad 2: GND -> DGND
- C52 pad 2: GND -> DGND
- C53 pad 2: GND -> DGND
- C54 pad 2: GND -> DGND
- C55 pad 2: GND -> DGND
- C56 pad 2: GND -> DGND
- C57 pad 2: GND -> DGND
- C58 pad 2: GND -> DGND
- C59 pad 2: GND -> DGND
- C6 pad 2: GND -> DGND
- C60 pad 2: GND -> DGND
- C61 pad 2: GND -> DGND
- C62 pad 2: GND -> DGND
- C63 pad 2: GND -> DGND
- C64 pad 2: GND -> DGND
- C65 pad 2: GND -> DGND
- C67 pad 1: GND -> DGND
- C68 pad 2: GND -> DGND
- C69 pad 2: GND -> DGND
- C7 pad 2: GND -> DGND
- C70 pad 2: GND -> DGND
- C72 pad 2: GND -> DGND
- C73 pad 2: GND -> DGND
- C78 pad 2: GND -> DGND
- C79 pad 2: GND -> DGND
- C8 pad 2: GND -> DGND
- C81 pad 2: GND -> DGND
- C82 pad 2: GND -> DGND
- C83 pad 2: GND -> DGND
- C84 pad 2: GND -> DGND
- C85 pad 2: GND -> DGND
- C86 pad 2: GND -> DGND
- C87 pad 2: GND -> DGND
- C88 pad 2: GND -> DGND
- C89 pad 2: GND -> DGND
- C9 pad 2: GND -> DGND
- C90 pad 1: JTAG_VCC -> Net-(C111-Pad1)
- C90 pad 2: GND -> DGND
- C91 pad 1: JTAG_VCC -> Net-(C111-Pad1)
- C91 pad 2: GND -> DGND
- C92 pad 2: GND -> DGND
- C93 pad 2: GND -> DGND
- C94 pad 2: GND -> DGND
- C95 pad 2: GND -> DGND
- C96 pad 2: GND -> DGND
- C97 pad 2: GND -> DGND
- C98 pad 2: GND -> DGND
- C99 pad 2: GND -> DGND
- D1 pad 1: Net-(C25-Pad1) -> Net-(D1-Pad1)
- D2 pad 2: GND -> DGND
- D3 pad 2: GND -> DGND
- D4 pad 1: GND -> DGND
- FB6 pad 2: Net-(FB6-Pad2) -> Net-(C111-Pad1)
- FL1 pad 4: GND -> DGND
- H1 pad 1: GND -> DGND
- H2 pad 1: GND -> DGND
- H3 pad 1: GND -> DGND
- J10 pad 2: GND -> DGND
- J12 pad 5: GND -> DGND
- J12 pad 6: GND -> DGND
- J13 pad 11: GND -> DGND
- J13 pad 6: GND -> DGND
- J14 pad 11: GND -> DGND
- J15 pad 4: GND -> DGND
- J15 pad 5: GND -> DGND
- J8 pad 6: GND -> DGND
- J9 pad 2: GND -> DGND
- JP1 pad 2: GND -> DGND
- JP2 pad 2: GND -> DGND
- JP3 pad 2: GND -> DGND
- JP4 pad 2: GND -> DGND
- JP5 pad 2: GND -> DGND
- L8 pad 2: GND -> DGND
- L9 pad 2: GND -> DGND
- LD1 pad 2: GND -> DGND
- LD11 pad 2: GND -> DGND
- LD12 pad 2: GND -> DGND
- LD2 pad 1: GND -> DGND
- LD2 pad 2: GND -> DGND
- LD2 pad 3: GND -> DGND
- LD3 pad 1: GND -> DGND
- LD3 pad 2: GND -> DGND
- LD3 pad 3: GND -> DGND
- LD4 pad 1: GND -> DGND
- LD4 pad 2: GND -> DGND
- LD4 pad 3: GND -> DGND
- LD5 pad 1: GND -> DGND
- LD5 pad 2: GND -> DGND
- LD5 pad 3: GND -> DGND
- LD6 pad 1: GND -> DGND
- LD6 pad 2: GND -> DGND
- LD6 pad 3: GND -> DGND
- LD7 pad 1: GND -> DGND
- LD7 pad 2: GND -> DGND
- LD7 pad 3: GND -> DGND
- LD8 pad 2: GND -> DGND
- LD9 pad 2: GND -> DGND
- Q11 pad 1: GND -> DGND
- Q12 pad 1: GND -> DGND
- Q13 pad 1: GND -> DGND
- Q2 pad 1: GND -> DGND
- Q4 pad 1: GND -> DGND
- Q5 pad 1: Net-(C25-Pad1) -> Net-(D1-Pad1)
- Q5 pad 2: Net-(C25-Pad1) -> Net-(D1-Pad1)
- Q5 pad 3: Net-(C25-Pad1) -> Net-(D1-Pad1)
- Q7 pad 1: GND -> DGND
- Q8 pad 1: /Power Supply/Stage 3 Regulators/1V8 Monitor/Vin -> Net-(C38-Pad1)
- Q8 pad 2: /Power Supply/Stage 3 Regulators/1V8 Monitor/Vin -> Net-(C38-Pad1)
- Q8 pad 3: /Power Supply/Stage 3 Regulators/1V8 Monitor/Vin -> Net-(C38-Pad1)
- Q9 pad 1: GND -> DGND
- Q9 pad 2: S3_PWR_ENABLE -> 1V8_IGood
- R110 pad 2: GND -> DGND
- R117 pad 1: GND -> DGND
- R121 pad 2: GND -> DGND
- R122 pad 2: GND -> DGND
- R136 pad 2: GND -> DGND
- R15 pad 2: GND -> DGND
- R16 pad 2: GND -> DGND
- R26 pad 2: GND -> DGND
- R27 pad 2: GND -> DGND
- R28 pad 2: GND -> DGND
- R38 pad 2: GND -> DGND
- R39 pad 2: GND -> DGND
- R40 pad 2: GND -> DGND
- R43 pad 2: GND -> DGND
- R45 pad 2: GND -> DGND
- R47 pad 2: GND -> DGND
- R55 pad 2: GND -> DGND
- R56 pad 2: GND -> DGND
- R57 pad 2: GND -> DGND
- R58 pad 1: /Power Supply/Stage 3 Regulators/1V8 Monitor/Vin -> Net-(C38-Pad1)
- R59 pad 1: /Power Supply/Stage 3 Regulators/1V8 Monitor/Vin -> Net-(C38-Pad1)
- R59 pad 2: /Power Supply/Stage 3 Regulators/1V8 Monitor/INa -> Net-(Q8-Pad4)
- R60 pad 1: /Power Supply/Stage 3 Regulators/1V8 Monitor/INa -> 3V3_LP
- R60 pad 2: /Power Supply/Stage 3 Regulators/1V8 Monitor/INb -> 1V8_IGood
- R62 pad 1: /Power Supply/Stage 3 Regulators/1V8 Monitor/INb -> DVDD
- R62 pad 2: GND -> /HDMI/VREF
- R63 pad 2: GND -> DGND
- R68 pad 2: GND -> DGND
- R69 pad 2: GND -> DGND
- R7 pad 2: GND -> DGND
- R70 pad 1: Net-(C40-Pad1) -> /HDMI/VREF
- R70 pad 2: 3V3_LP -> DGND
- R71 pad 1: /Power Supply/Stage 3 Regulators/1V8 Monitor/Vin -> DVDD
- R71 pad 2: Net-(Q8-Pad4) -> Net-(R71-Pad2)
- R72 pad 1: Net-(C40-Pad1) -> Net-(LD13-Pad2)
- R72 pad 2: 1V8_V_Good -> ~VDMA_Lock
- R73 pad 1: 3V3_LP -> Net-(LD13-Pad3)
- R73 pad 2: 1V8_I_Good -> ~VDMA_Underflow
- R8 pad 2: GND -> DGND
- R85 pad 2: GND -> DGND
- R86 pad 2: GND -> DGND
- R87 pad 2: GND -> DGND
- SW2 pad 3: GND -> DGND
- SW2 pad 4: GND -> DGND
- T1 pad 3: GND -> DGND
- U1 pad 8: GND -> DGND
- U10 pad 1: GND -> DGND
- U11 pad 1: 1V8_I_Good -> 1V8_IGood
- U11 pad 5: GND -> DGND
- U11 pad 8: Net-(R75-Pad2) -> DGND
- U11 pad 9: Net-(R74-Pad2) -> DGND
- U12 pad 1: 1V8_V_Good -> DVDD
- U12 pad 2: GND -> /HDMI/Active
- U12 pad 3: /Power Supply/Stage 3 Regulators/1V8 Monitor/INa -> /HDMI/VREF
- U12 pad 4: /Power Supply/Stage 3 Regulators/1V8 Monitor/INb -> /HDMI/HSync
- U12 pad 5: Net-(C40-Pad1) -> /HDMI/VSync
- U12 pad 6: 1V8_V_Good -> Net-(U12-Pad6)
- U13 pad 5: GND -> DGND
- U14 pad 2: GND -> DGND
- U15 pad 49: GND -> DGND
- U16 pad 4: GND -> DGND
- U17 pad 10: GND -> DGND
- U17 pad 11: GND -> DGND
- U17 pad 14: GND -> DGND
- U17 pad 18: GND -> DGND
- U17 pad 2: GND -> DGND
- U17 pad 31: GND -> DGND
- U17 pad 4: GND -> DGND
- U17 pad 50: GND -> DGND
- U17 pad 61: GND -> DGND
- U17 pad 65: GND -> DGND
- U17 pad 7: GND -> DGND
- U18 pad 1.1: GND -> DGND
- U18 pad 1.19: GND -> DGND
- U18 pad 1.25: GND -> DGND
- U18 pad 1.30: GND -> DGND
- U18 pad 1.33: GND -> DGND
- U18 pad 1.43: GND -> DGND
- U18 pad 1.53: GND -> DGND
- U18 pad 1.54: GND -> DGND
- U18 pad 1.63: GND -> DGND
- U18 pad 1.64: GND -> DGND
- U18 pad 1.7: GND -> DGND
- U18 pad 1.73: GND -> DGND
- U18 pad 1.74: GND -> DGND
- U18 pad 1.83: GND -> DGND
- U18 pad 1.89: GND -> DGND
- U18 pad 2.19: GND -> DGND
- U18 pad 2.29: GND -> DGND
- U18 pad 2.30: GND -> DGND
- U18 pad 2.39: GND -> DGND
- U18 pad 2.40: GND -> DGND
- U18 pad 2.49: GND -> DGND
- U18 pad 2.50: GND -> DGND
- U18 pad 2.59: GND -> DGND
- U18 pad 2.60: GND -> DGND
- U18 pad 2.61: Net-(U18-Pad2.61) -> HDMI_R3
- U18 pad 2.63: Net-(U18-Pad2.63) -> HDMI_R2
- U18 pad 2.65: Net-(U18-Pad2.65) -> HDMI_R1
- U18 pad 2.67: Net-(U18-Pad2.67) -> HDMI_R0
- U18 pad 2.69: GND -> DGND
- U18 pad 2.70: GND -> DGND
- U18 pad 2.71: Net-(U18-Pad2.71) -> HDMI_G3
- U18 pad 2.73: Net-(U18-Pad2.73) -> HDMI_G2
- U18 pad 2.75: Net-(U18-Pad2.75) -> HDMI_G1
- U18 pad 2.77: Net-(U18-Pad2.77) -> HDMI_G0
- U18 pad 2.79: GND -> DGND
- U18 pad 2.80: GND -> DGND
- U18 pad 2.81: Net-(U18-Pad2.81) -> HDMI_B3
- U18 pad 2.83: Net-(U18-Pad2.83) -> HDMI_B2
- U18 pad 2.85: Net-(U18-Pad2.85) -> HDMI_CLK
- U18 pad 2.87: Net-(U18-Pad2.87) -> HDMI_B1
- U18 pad 2.88: Net-(U18-Pad2.88) -> ~VDMA_Underflow
- U18 pad 2.89: GND -> DGND
- U18 pad 2.90: Net-(U18-Pad2.90) -> ~VDMA_Lock
- U18 pad 2.91: Net-(U18-Pad2.91) -> HDMI_B0
- U18 pad 2.92: JTAG_VCC -> Net-(U18-Pad2.92)
- U18 pad 2.93: Net-(U18-Pad2.93) -> HDMI_Active
- U18 pad 2.95: Net-(U18-Pad2.95) -> HDMI_HSync
- U18 pad 2.97: Net-(U18-Pad2.97) -> HDMI_VSync
- U18 pad 3.11: GND -> DGND
- U18 pad 3.12: GND -> DGND
- U18 pad 3.17: GND -> DGND
- U18 pad 3.18: GND -> DGND
- U18 pad 3.23: GND -> DGND
- U18 pad 3.24: GND -> DGND
- U18 pad 3.29: GND -> DGND
- U18 pad 3.30: GND -> DGND
- U18 pad 3.35: GND -> DGND
- U18 pad 3.36: GND -> DGND
- U18 pad 3.45: GND -> DGND
- U18 pad 3.46: GND -> DGND
- U18 pad 3.5: GND -> DGND
- U18 pad 3.55: GND -> DGND
- U18 pad 3.6: GND -> DGND
- U18 pad SH1: GND -> DGND
- U18 pad SH2: GND -> DGND
- U18 pad SH3: GND -> DGND
- U19 pad 1: GND -> DGND
- U19 pad 14: GND -> DGND
- U19 pad 15: Net-(FB6-Pad2) -> Net-(C111-Pad1)
- U19 pad 7: GND -> DGND
- U19 pad 8: JTAG_VCC -> Net-(C111-Pad1)
- U2 pad 5: GND -> DGND
- U20 pad 2: GND -> DGND
- U21 pad 11: GND -> DGND
- U21 pad 2: GND -> DGND
- U21 pad 24: GND -> Net-(R142-Pad1)
- U21 pad 25: GND -> DGND
- U22 pad 2: GND -> DGND
- U23 pad 2: GND -> DGND
- U24 pad 17: GND -> DGND
- U24 pad 2: GND -> DGND
- U3 pad 2: GND -> DGND
- U4 pad 8: GND -> DGND
- U5 pad 5: GND -> DGND
- U6 pad 2: GND -> DGND
- U7 pad 1: GND -> DGND
- U8 pad 5: GND -> DGND
- U9 pad 2: GND -> DGND
- Y1 pad 2: GND -> DGND
Routing:
- net GND: track 919.7 -> 0.00 mm, vias 612 -> 6
- net DGND: track 0.00 -> 844.3 mm, vias 0 -> 591
- net JTAG_TMS: track 0.00 -> 82.4 mm, vias 0 -> 2
- net JTAG_TDO: track 0.00 -> 80.2 mm, vias 0 -> 2
- net JTAG_TDI: track 0.00 -> 80.0 mm, vias 0 -> 2
- net JTAG_TCK: track 0.00 -> 79.8 mm, vias 0 -> 2
- net ~VDMA_Underflow: track 0.00 -> 65.8 mm, vias 0 -> 2
- net /Power Supply/Stage 2 Regulators/5V_5A Regulator/Vout: track 79.1 -> 15.7 mm
- net ~VDMA_Lock: track 0.00 -> 62.9 mm, vias 0 -> 2
- net DVDD: track 0.00 -> 59.3 mm, vias 0 -> 6
- net 1V8_from_FPGA: track 3.85 -> 52.3 mm, vias 2 -> 0
- net /HDMI/R3: track 0.00 -> 40.7 mm
- net /HDMI/R2: track 0.00 -> 39.0 mm
- net /Power Supply/Stage 2 Regulators/5V_5A Regulator/FB_Gnd: track 48.0 -> 9.59 mm
- net HDMI_VSync: track 0.00 -> 37.4 mm
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- added copper zone on In2.Cu, net +3V3
- added copper zone on B.Cu, net DGND
- added copper zone on F.Cu, net DGND
- added copper zone on In1.Cu, net DGND
- added copper zone on F.Cu, net Net-(C38-Pad1)
- added copper zone on F.Cu, net Net-(D1-Pad1)
- removed copper zone on F.Cu, net /Power Supply/Stage 3 Regulators/1V8 Monitor/Vin
- removed copper zone on B.Cu, net GND
- removed copper zone on F.Cu, net GND
- removed copper zone on In1.Cu, net GND
Other:
- board size 206 x 145 mm -> 200 x 150 mm
- net class USB: clearance 0.2 -> 0.0889
- board text added: "<- No coffee before soldering these"
- board text added: "VDMA"
- board text removed: "+"
- board text removed: "3V3_LP"
- board text removed: "Battery"
- board text removed: "No coffee before soldering these ->"

Commit message: mostly tidying up stuff that was laid out too quickly at the weekend
Parts:
- added H10: MountingHole_Pad, MountingHole:MountingHole_3.2mm_M3_Pad_Via, F.Cu at (52.5, 111.0)
- added H11: MountingHole_Pad, MountingHole:MountingHole_3.2mm_M3_Pad_Via, F.Cu at (256.5, 89.0)
- added H12: MountingHole_Pad, MountingHole:MountingHole_3.2mm_M3_Pad_Via, F.Cu at (242.5, 96.0)
- added H4: MountingHole_Pad, MountingHole:MountingHole_3.2mm_M3_Pad_Via, F.Cu at (75.5, 32.0)
- added H5: MountingHole_Pad, MountingHole:MountingHole_3.2mm_M3_Pad_Via, F.Cu at (111.5, 48.0)
- added H6: MountingHole_Pad, MountingHole:MountingHole_3.2mm_M3_Pad_Via, F.Cu at (241.5, 30.0)
- added H7: MountingHole_Pad, MountingHole:MountingHole_3.2mm_M3_Pad_Via, F.Cu at (52.5, 171.0)
- added H8: MountingHole_Pad, MountingHole:MountingHole_3.2mm_M3_Pad_Via, F.Cu at (165.5, 171.0)
- added H9: MountingHole_Pad, MountingHole:MountingHole_3.2mm_M3_Pad_Via, F.Cu at (242.5, 171.0)
- RN5, RN6: footprint Resistor_SMD:R_Cat16-8 -> Resistor_SMD:R_Array_Convex_8x0602
- moved LD6 294.0 mm to (92.8, 67.0), turned to 270 degrees
- moved R102 290.9 mm to (91.2, 73.0), turned to 90 degrees
- moved R101 289.2 mm to (92.8, 73.0), turned to 90 degrees
- moved H3 289.0 mm to (-119.8, 75.5)
- moved LD5 288.1 mm to (97.8, 67.0), turned to 270 degrees
- moved C13 287.8 mm to (-142.5, 82.5)
- moved C14 287.8 mm to (-131.0, 82.5)
- moved C15 287.8 mm to (-127.2, 82.5)
- moved C16 287.8 mm to (-118.0, 88.8)
- moved C17 287.8 mm to (-111.8, 82.5)
- moved C18 287.8 mm to (-107.8, 82.5)
- moved C19 287.8 mm to (-100.8, 80.2)
- moved L2 287.8 mm to (-136.8, 82.5)
- moved R10 287.8 mm to (-114.8, 86.5)
- moved R11 287.8 mm to (-118.0, 86.5)
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Connections:
- J8 pad 2: /Power Supply/Power Rail Management/12V_VFault -> /Power Supply/Power Rail Management/3V3ADC_VFault
- J8 pad 3: /Power Supply/Power Rail Management/12V_OK -> /Power Supply/Power Rail Management/3V3ADC_OK
- J8 pad 4: /Power Supply/Power Rail Management/12V_IFault -> /Power Supply/Power Rail Management/3V3ADC_IFault
- J8 pad 5: /Power Supply/Power Rail Management/3V3_VFault -> /Power Supply/Power Rail Management/1V8_VFault
- R100 pad 1: /Power Supply/Power Rail Management/3V3ADC_VFault -> /Power Supply/Power Rail Management/12V_VFault
- R101 pad 1: /Power Supply/Power Rail Management/3V3ADC_OK -> /Power Supply/Power Rail Management/12V_OK
- R102 pad 1: /Power Supply/Power Rail Management/3V3ADC_IFault -> /Power Supply/Power Rail Management/12V_IFault
- R88 pad 1: /Power Supply/Power Rail Management/12V_VFault -> /Power Supply/Power Rail Management/3V3ADC_VFault
- R89 pad 1: /Power Supply/Power Rail Management/12V_OK -> /Power Supply/Power Rail Management/3V3ADC_OK
- R90 pad 1: /Power Supply/Power Rail Management/12V_IFault -> /Power Supply/Power Rail Management/3V3ADC_IFault
- R91 pad 1: /Power Supply/Power Rail Management/3V3_VFault -> /Power Supply/Power Rail Management/1V8_VFault
- R92 pad 1: /Power Supply/Power Rail Management/3V3_OK -> /Power Supply/Power Rail Management/1V8_OK
- R93 pad 1: /Power Supply/Power Rail Management/3V3_IFault -> /Power Supply/Power Rail Management/1V8_IFault
- R97 pad 1: /Power Supply/Power Rail Management/1V8_VFault -> /Power Supply/Power Rail Management/3V3_VFault
- R98 pad 1: /Power Supply/Power Rail Management/1V8_OK -> /Power Supply/Power Rail Management/3V3_OK
- R99 pad 1: /Power Supply/Power Rail Management/1V8_IFault -> /Power Supply/Power Rail Management/3V3_IFault
- U15 pad 10: /Power Supply/Power Rail Management/1V8_IFault -> /Power Supply/Power Rail Management/3V3_IFault
- U15 pad 11: /Power Supply/Power Rail Management/3V3ADC_VFault -> /Power Supply/Power Rail Management/12V_VFault
- U15 pad 12: /Power Supply/Power Rail Management/3V3ADC_OK -> /Power Supply/Power Rail Management/12V_OK
- U15 pad 14: /Power Supply/Power Rail Management/3V3ADC_IFault -> /Power Supply/Power Rail Management/12V_IFault
- U15 pad 15: /Power Supply/Power Rail Management/16V_VFault -> S3_PWR_ENABLE
- U15 pad 16: 16V_OK -> S2_PWR_ENABLE
- U15 pad 17: /Power Supply/Power Rail Management/16V_IFault -> /Power Supply/Power Rail Management/UART_Error
- U15 pad 18: UART_PMIC_TO_FPGA -> S1_PWR_ENABLE
- U15 pad 19: UART_PMIC_FROM_FPGA -> /Power Supply/Power Rail Management/I2C_Error
- U15 pad 2: /Power Supply/Power Rail Management/3V3_OK -> /Power Supply/Power Rail Management/1V8_OK
- U15 pad 20: 12V_I_Good -> UART_PMIC_TO_FPGA
- U15 pad 21: 12V_V_Good -> UART_PMIC_FROM_FPGA
- U15 pad 23: 3V3_I_Good -> 12V_I_Good
- U15 pad 24: 3V3_V_Good -> 12V_V_Good
- U15 pad 26: 5V_I_Good -> 3V3_I_Good
- U15 pad 27: 5V_V_Good -> 3V3_V_Good
- U15 pad 28: 1V8_I_Good -> 5V_I_Good
- U15 pad 29: 1V8_V_Good -> 5V_V_Good
- U15 pad 3: /Power Supply/Power Rail Management/3V3_IFault -> /Power Supply/Power Rail Management/1V8_IFault
- U15 pad 31: 3V3ADC_I_Good -> 1V8_I_Good
- U15 pad 32: 3V3ADC_V_Good -> 1V8_V_Good
- U15 pad 33: FPGA_PWR_GOOD -> 3V3ADC_I_Good
- U15 pad 34: Net-(U15-Pad34) -> 3V3ADC_V_Good
- U15 pad 35: S3_PWR_ENABLE -> FPGA_PWR_GOOD
- U15 pad 36: S2_PWR_ENABLE -> Net-(U15-Pad36)
- U15 pad 37: /Power Supply/Power Rail Management/UART_Error -> Net-(U15-Pad37)
- U15 pad 38: S1_PWR_ENABLE -> Net-(U15-Pad38)
- U15 pad 40: /Power Supply/Power Rail Management/I2C_Error -> Net-(U15-Pad40)
- U15 pad 44: /Power Supply/Power Rail Management/12V_VFault -> /Power Supply/Power Rail Management/3V3ADC_VFault
- U15 pad 45: /Power Supply/Power Rail Management/12V_OK -> /Power Supply/Power Rail Management/3V3ADC_OK
- U15 pad 47: /Power Supply/Power Rail Management/12V_IFault -> /Power Supply/Power Rail Management/3V3ADC_IFault
- U15 pad 48: /Power Supply/Power Rail Management/3V3_VFault -> /Power Supply/Power Rail Management/1V8_VFault
- U15 pad 8: /Power Supply/Power Rail Management/1V8_VFault -> /Power Supply/Power Rail Management/3V3_VFault
- U15 pad 9: /Power Supply/Power Rail Management/1V8_OK -> /Power Supply/Power Rail Management/3V3_OK
Routing:
- net +1V8: track 18.3 -> 68.9 mm, vias 5 -> 6
- net Net-(C97-Pad1): track 0.00 -> 36.4 mm
- net /HDMI/B0: track 11.6 -> 46.4 mm
- net /HDMI/B3: track 15.5 -> 50.2 mm
- net /HDMI/B1: track 12.5 -> 47.1 mm
- net /HDMI/Clk: track 13.4 -> 47.8 mm
- net /HDMI/B2: track 14.6 -> 48.8 mm
- net /HDMI/G0: track 27.6 -> 61.2 mm
- net /Power Supply/Power Rail Management/I2C_Error: track 12.7 -> 46.2 mm
- net /HDMI/G1: track 29.2 -> 62.6 mm
- net HDMI_VSync: track 37.4 -> 4.10 mm
- net /HDMI/VSync: track 7.22 -> 40.5 mm
- net HDMI_HSync: track 37.3 -> 4.05 mm
- net /HDMI/G2: track 30.9 -> 64.1 mm
- net /HDMI/HSync: track 7.34 -> 40.5 mm
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- added copper zone on In2.Cu, net DGND
Other:
- board text removed: "OFF"
