File: v1.kicad_pcb (KiCad board)
At the start: 4 copper layers, 200 x 150 mm, 380 parts, among them J1 Powerpole G1377G2, J10 Conn_Coaxial, J12 USB_B_Micro, J13 Micro_SD_Card_Det, J14 ARJM11D7-502-AB-EW2, J15 USB_A, J17 HDMI_A, J2 Barrel_Jack, J3 Conn_01x02, J4 Conn_01x02, J5 Conn_01x02, J6 Conn_01x02, J7 Conn_01x02, J8 Conn_01x06_Male, J9 Conn_Coaxial, M1 Logo_10mmx10mm, Q1 Si7141DP, Q10 Si7141DP, Q11 SI1539CDL-T1-GE3, Q12 SI1539CDL-T1-GE3, Q13 SI1539CDL-T1-GE3, Q2 SI1539CDL-T1-GE3, Q3 Si7141DP, Q4 SI1539CDL-T1-GE3, Q5 Si7141DP, Q6 Si7141DP, Q7 SI1539CDL-T1-GE3, Q8 Si7141DP, Q9 SI1539CDL-T1-GE3, SW1 SW_SPDT, SW2 Tactile_Switch_Generic, T1 PWB2010L, T2 Macom_ETC1-1-13, U1 171050601, U10 NCP1117-3.3_TO252, U11 MAX9612, U12 TFP410PAP, U13 MAX9612, U14 TPS3701DDCR, U15 LCMXO2-640HC-4SG48C, U16 REF5025IDGK, U17 LTC2216, U18 TE0720, U19 JTAG-SMT3, U2 MAX9612, U20 TPD2S017, U21 TXS02612, U22 TPS2051B, U23 TPD2S017, U24 AD5689RxCPZ, U3 TPS3701DDCR, U4 171050601, U5 MAX9612, U6 TPS3701DDCR, U7 NCP1117-3.3_TO252, U8 MAX9612, U9 TPS3701DDCR, Y1 SIT5001AC-3E-33N0-80.000000X

Commit message: layout getting there! :)
Parts:
- removed the C35 at (226.0, 118.0)
- removed the H2 at (-119.5, 119.2)
- added C112: 100n, Capacitor_SMD:C_0603_1608Metric, F.Cu at (122.0, 93.8)
- added C113: 100n, Capacitor_SMD:C_0603_1608Metric, F.Cu at (107.5, 93.8)
- added C114: 100n, Capacitor_SMD:C_0603_1608Metric, F.Cu at (93.0, 93.8)
- added C115: 100n, Capacitor_SMD:C_0603_1608Metric, F.Cu at (78.5, 93.8)
- added C116: 100n, Capacitor_SMD:C_0603_1608Metric, F.Cu at (64.0, 93.8)
- added C39: 4u7, Capacitor_SMD:C_0603_1608Metric, F.Cu at (238.8, 106.0)
- added H10: Shield, Shield_WUT:Shield_Masach_MS570-10_52.7x30.7x6mm_TH, F.Cu at (147.8, 135.5)
- added LD14: ACDA02-41SURKWA-F01, Display_WUT:ACDA02-41SURKWA-F01, F.Cu at (122.0, 107.8)
- added LD15: ACDA02-41SURKWA-F01, Display_WUT:ACDA02-41SURKWA-F01, F.Cu at (107.5, 107.8)
- added LD16: ACDA02-41SURKWA-F01, Display_WUT:ACDA02-41SURKWA-F01, F.Cu at (93.0, 107.8)
- added LD17: ACDA02-41SURKWA-F01, Display_WUT:ACDA02-41SURKWA-F01, F.Cu at (78.5, 107.8)
- added LD18: ACDA02-41SURKWA-F01, Display_WUT:ACDA02-41SURKWA-F01, F.Cu at (64.0, 107.8)
- added R138: 22k, Resistor_SMD:R_0603_1608Metric, F.Cu at (122.0, 92.0)
- added R139: 22k, Resistor_SMD:R_0603_1608Metric, F.Cu at (107.5, 92.0)
- added R140: 22k, Resistor_SMD:R_0603_1608Metric, F.Cu at (93.0, 92.0)
- added R141: 22k, Resistor_SMD:R_0603_1608Metric, F.Cu at (78.5, 92.0)
- added R142: 22k, Resistor_SMD:R_0603_1608Metric, F.Cu at (64.0, 92.0)
- added U26: TLC59281RGER, Package_DFN_QFN:QFN-24-1EP_4x4mm_P0.5mm_EP2.6x2.6mm, F.Cu at (122.0, 97.2)
- added U28: TLC59281RGER, Package_DFN_QFN:QFN-24-1EP_4x4mm_P0.5mm_EP2.6x2.6mm, F.Cu at (107.5, 97.2)
- added U30: TLC59281RGER, Package_DFN_QFN:QFN-24-1EP_4x4mm_P0.5mm_EP2.6x2.6mm, F.Cu at (93.0, 97.2)
- added U32: TLC59281RGER, Package_DFN_QFN:QFN-24-1EP_4x4mm_P0.5mm_EP2.6x2.6mm, F.Cu at (78.5, 97.2)
- added U34: TLC59281RGER, Package_DFN_QFN:QFN-24-1EP_4x4mm_P0.5mm_EP2.6x2.6mm, F.Cu at (64.0, 97.2)
- C19, C7: footprint Capacitor_WUT:Wurth_WCAP_PSHP -> Capacitor_WUT:Wurth_WCAP_PSLP
- J2: value Barrel_Jack -> Barrel_Jack_Switch
- M1: value Logo_10mmx10mm -> Logo_16mmx16mm; footprint Misc_WUT:Logo_10mmx10mm -> Misc_WUT:Logo_16mmx16mm
- moved H11 333.2 mm to (209.2, 128.5)
- moved C13 328.9 mm to (184.0, 122.5)
- moved L2 326.0 mm to (186.0, 128.5)
- moved C14 322.0 mm to (188.5, 122.5)
- moved C17 319.5 mm to (204.8, 126.0)
- moved C18 319.5 mm to (208.8, 126.0)
- moved C15 319.3 mm to (187.8, 134.5), turned to 270 degrees
- moved C16 319.0 mm to (197.8, 134.2)
- moved R10 319.0 mm to (201.0, 132.0)
- moved R11 319.0 mm to (197.8, 132.0)
- moved R29 319.0 mm to (191.2, 132.0)
- moved R30 319.0 mm to (194.5, 132.0)
- moved R31 319.0 mm to (194.5, 134.2)
- moved U4 319.0 mm to (196.2, 121.0)
- moved C19 312.2 mm to (206.8, 134.5), turned to 90 degrees
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- renumbered C42 to C102, C110 to C103, C102 to C104, C103 to C105, C104 to C106, C105 to C107, C106 to C108, C107 to C109, C108 to C110, C109 to C111, C38 to C35, C39 to C36, C40 to C37, C41 to C38, C36 to C40, C37 to C41, C43 to C42, C44 to C43, C45 to C44, C46 to C45, C47 to C46, C49 to C48, C50 to C49, C51 to C50, C52 to C51, C53 to C52, C54 to C53, C55 to C54, C56 to C55, C57 to C56, C58 to C57, C59 to C58, C60 to C59, C61 to C60, C62 to C61, C63 to C62, C64 to C63, C65 to C64, C66 to C65, C67 to C66, C68 to C67, C69 to C68, C70 to C69, C71 to C70, C72 to C71, C73 to C72, C74 to C73, C75 to C74, C76 to C75, C77 to C76, C78 to C77, C79 to C78, C80 to C79, C81 to C80, C82 to C81, C83 to C82, C84 to C83, C85 to C84, C86 to C85, C87 to C86, C88 to C87, C89 to C88, C90 to C89, C91 to C90, C111 to C91, H4 to H1, H3 to H11, H1 to H12, H5 to H2, H6 to H3, H7 to H4, H8 to H5, H9 to H6, H10 to H7, H11 to H8, H12 to H9, J12 to J11, J13 to J12, J14 to J13, J15 to J14, J17 to J15, L9 to L10, L10 to L3, L3 to L4, L4 to L5, L5 to L6, L6 to L7, L7 to L8, L8 to L9, R110 to R100, R111 to R101, R112 to R102, R113 to R103, R114 to R104, R115 to R105, R116 to R106, R117 to R107, R118 to R108, R119 to R109, R120 to R110, R121 to R111, R122 to R112, R123 to R113, R124 to R114, R125 to R115, R126 to R116, R127 to R117, R128 to R118, R129 to R119, R130 to R120, R131 to R121, R132 to R122, R133 to R123, R134 to R124, R135 to R125, R136 to R126, R142 to R127, R137 to R128, R138 to R129, R139 to R130, R140 to R131, R141 to R132, R62 to R133, R70 to R134, R71 to R135, R72 to R136, R73 to R137, R63 to R62, R64 to R63, R65 to R64, R66 to R65, R67 to R66, R68 to R67, R69 to R68, R79 to R69, R80 to R70, R81 to R71, R82 to R72, R83 to R73, R84 to R74, R85 to R75, R86 to R76, R87 to R77, R88 to R78, R89 to R79, R90 to R80, R91 to R81, R92 to R82, R93 to R83, R94 to R84, R95 to R85, R96 to R86, R97 to R87, R98 to R88, R99 to R89, R100 to R90, R101 to R91, R102 to R92, R103 to R93, R104 to R94, R105 to R95, R106 to R96, R107 to R97, R108 to R98, R109 to R99, U11 to U10, U10 to U11, U13 to U12, U14 to U13, U15 to U14, U16 to U15, U17 to U16, U18 to U17, U19 to U18, U20 to U19, U21 to U20, U22 to U21, U23 to U22, U24 to U23, U12 to U24
Connections:
- J2 pad 3: (no net) -> Net-(FL1-Pad3)
- U24 pad 10: Net-(U12-Pad10) -> DVDD
- U24 pad 35: DVDD -> DGND
Routing:
- net +3V3: track 81.4 -> 156.2 mm, vias 36 -> 75
- net DGND: track 852.3 -> 904.2 mm, vias 590 -> 642
- net /Power Supply/Stage 2 Regulators/12V_In: track 37.7 -> 14.4 mm, vias 4 -> 7
- net MON_SCL: track 5.18 -> 27.7 mm, vias 0 -> 3
- net MON_SDA: track 6.57 -> 28.1 mm, vias 0 -> 3
- net /User Interface/Dual Seven Segment Display 5/D2_DP: track 0.00 -> 19.3 mm
- net /User Interface/Dual Seven Segment Display 4/D2_DP: track 0.00 -> 19.3 mm
- net /User Interface/Dual Seven Segment Display 3/D2_DP: track 0.00 -> 19.3 mm
- net /User Interface/Dual Seven Segment Display 2/D2_DP: track 0.00 -> 19.3 mm
- net /User Interface/Dual Seven Segment Display 1/D2_DP: track 0.00 -> 19.3 mm
- net /User Interface/Dual Seven Segment Display 4/D1_E: track 0.00 -> 18.7 mm
- net /User Interface/Dual Seven Segment Display 3/D1_E: track 0.00 -> 18.7 mm
- net /User Interface/Dual Seven Segment Display 2/D1_E: track 0.00 -> 18.7 mm
- net /User Interface/Dual Seven Segment Display 1/D1_E: track 0.00 -> 18.7 mm
- net /User Interface/Dual Seven Segment Display 5/D1_E: track 0.00 -> 18.7 mm
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- added copper zone on In2.Cu, net +5V
- added copper zone on In2.Cu, net /Power Supply/Stage 2 Regulators/12V_In
- added copper zone on In2.Cu, net 3V3_LP
- added copper zone on F.Cu, net Net-(C40-Pad1)

Commit message: broke many things in the name of progress. Restore point = this commit - 1
Parts:
- removed R134: 10k, Resistor_SMD:R_0603_1608Metric
- added C117: 22u, Capacitor_SMD:C_1210_3225Metric, F.Cu at (237.0, 134.8)
- added C118: 1u, Capacitor_SMD:C_0603_1608Metric, F.Cu at (240.0, 143.2)
- added C119: 100n, Capacitor_SMD:C_0402_1005Metric, F.Cu at (12.5, -2.25)
- added C120: 47p, Capacitor_SMD:C_0402_1005Metric, F.Cu at (15.4, -2.25)
- added C121: 150p, Capacitor_SMD:C_0402_1005Metric, F.Cu at (12.5, -0.26)
- added C122: 47p, Capacitor_SMD:C_0402_1005Metric, F.Cu at (12.5, 1.73)
- added J16: Conn_Coaxial, Connector_WUT:SMA_Linx_CONSMA002-L-G_Horizontal, F.Cu at (6.67, 5.20)
- added L11: 330n, Inductor_SMD:L_0805_2012Metric, F.Cu at (22.0, -9.89)
- added L12: 330n, Inductor_SMD:L_0805_2012Metric, F.Cu at (22.0, -6.94)
- added REF**: Shield_Masach_MS570-10_52.7x30.7x6mm_TH, Shield_WUT:Shield_Masach_MS570-10_52.7x30.7x6mm_TH, F.Cu at (217.2, 101.6)
- added T3: PWB2010L, Transformer_WUT:Coilcraft_PWB, F.Cu at (37.8, 17.0)
- added U25: AD9744_LFCSP, Package_CSP:LFCSP-32-1EP_5x5mm_P0.5mm_EP3.25x3.25mm, F.Cu at (28.0, 17.0)
- C39, C40: value 4u7 -> 22u; footprint Capacitor_SMD:C_0603_1608Metric -> Capacitor_SMD:C_1210_3225Metric
- R133: value 27k -> 0
- U11: value NCP1117-3.3_TO252 -> ADM7154; footprint Package_TO_SOT_SMD:TO-252-2 -> Package_CSP:LFCSP-8-1EP_3x3mm_P0.5mm_EP1.45x1.74mm
- U23: value AD5689RxCPZ -> AD5689BCPZ
- moved C25 408.5 mm to (-236.6, 173.3)
- moved C26 408.5 mm to (-224.8, 168.1)
- moved C27 408.5 mm to (-236.4, 142.4)
- moved C28 408.5 mm to (-241.7, 147.2)
- moved C29 408.5 mm to (-233.9, 132.8)
- moved C30 408.5 mm to (-290.3, 175.6)
- moved C31 408.5 mm to (-287.8, 176.6)
- moved C32 408.5 mm to (-289.8, 160.3)
- moved C33 408.5 mm to (-251.2, 174.6)
- moved C34 408.5 mm to (-269.6, 175.3)
- moved D1 408.5 mm to (-228.2, 168.4)
- moved D2 408.5 mm to (-216.5, 165.8)
- moved D3 408.5 mm to (-234.2, 136.7)
- moved F1 408.5 mm to (-232.4, 140.9)
- moved FL1 408.5 mm to (-213.3, 157.9)
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Connections:
- C1 pad 2: DGND -> ACOM
- C10 pad 2: DGND -> ACOM
- C100 pad 2: DGND -> ACOM
- C101 pad 2: DGND -> ACOM
- C102 pad 2: DGND -> ACOM
- C103 pad 2: DGND -> ACOM
- C104 pad 2: DGND -> ACOM
- C105 pad 2: DGND -> ACOM
- C106 pad 2: DGND -> ACOM
- C107 pad 2: DGND -> ACOM
- C108 pad 2: DGND -> ACOM
- C109 pad 2: DGND -> ACOM
- C11 pad 2: DGND -> ACOM
- C110 pad 2: DGND -> ACOM
- C111 pad 2: DGND -> ACOM
- C112 pad 2: DGND -> ACOM
- C113 pad 2: DGND -> ACOM
- C114 pad 2: DGND -> ACOM
- C115 pad 2: DGND -> ACOM
- C116 pad 2: DGND -> ACOM
- C12 pad 2: DGND -> ACOM
- C13 pad 2: DGND -> ACOM
- C14 pad 2: DGND -> ACOM
- C15 pad 2: DGND -> ACOM
- C17 pad 2: DGND -> ACOM
- C18 pad 2: DGND -> ACOM
- C19 pad 2: DGND -> ACOM
- C2 pad 2: DGND -> ACOM
- C20 pad 2: DGND -> ACOM
- C21 pad 2: DGND -> ACOM
- C22 pad 2: DGND -> ACOM
- C23 pad 2: DGND -> ACOM
- C24 pad 2: DGND -> ACOM
- C25 pad 2: DGND -> ACOM
- C26 pad 2: DGND -> ACOM
- C27 pad 2: DGND -> ACOM
- C28 pad 2: DGND -> ACOM
- C29 pad 2: DGND -> ACOM
- C3 pad 2: DGND -> ACOM
- C30 pad 2: DGND -> ACOM
- C31 pad 2: DGND -> ACOM
- C32 pad 2: DGND -> ACOM
- C33 pad 2: DGND -> ACOM
- C34 pad 2: DGND -> ACOM
- C35 pad 2: DGND -> ACOM
- C36 pad 2: DGND -> ACOM
- C37 pad 2: DGND -> ACOM
- C38 pad 2: DGND -> ACOM
- C39 pad 2: DGND -> ACOM
- C40 pad 2: DGND -> ACOM
- C41 pad 1: Net-(C40-Pad1) -> Net-(C41-Pad1)
- C41 pad 2: DGND -> ACOM
- C42 pad 2: DGND -> ACOM
- C43 pad 2: DGND -> ACOM
- C44 pad 2: DGND -> ACOM
- C45 pad 2: DGND -> ACOM
- C46 pad 2: DGND -> ACOM
- C48 pad 2: DGND -> ACOM
- C49 pad 2: DGND -> ACOM
- C5 pad 2: DGND -> ACOM
- C50 pad 2: DGND -> ACOM
- C51 pad 2: DGND -> ACOM
- C52 pad 2: DGND -> ACOM
- C53 pad 2: DGND -> ACOM
- C54 pad 2: DGND -> ACOM
- C55 pad 2: DGND -> ACOM
- C56 pad 2: DGND -> ACOM
- C57 pad 2: DGND -> ACOM
- C58 pad 2: DGND -> ACOM
- C59 pad 2: DGND -> ACOM
- C6 pad 2: DGND -> ACOM
- C60 pad 2: DGND -> ACOM
- C61 pad 2: DGND -> ACOM
- C62 pad 2: DGND -> ACOM
- C63 pad 2: DGND -> ACOM
- C64 pad 2: DGND -> ACOM
- C66 pad 1: DGND -> ACOM
- C67 pad 2: DGND -> ACOM
- C68 pad 2: DGND -> ACOM
- C69 pad 2: DGND -> ACOM
- C7 pad 2: DGND -> ACOM
- C71 pad 2: DGND -> ACOM
- C72 pad 2: DGND -> ACOM
- C77 pad 2: DGND -> ACOM
- C78 pad 2: DGND -> ACOM
- C8 pad 2: DGND -> ACOM
- C80 pad 2: DGND -> ACOM
- C81 pad 2: DGND -> ACOM
- C82 pad 2: DGND -> ACOM
- C83 pad 2: DGND -> ACOM
- C84 pad 2: DGND -> ACOM
- C85 pad 2: DGND -> ACOM
- C86 pad 2: DGND -> ACOM
- C87 pad 2: DGND -> ACOM
- C88 pad 2: DGND -> ACOM
- C89 pad 2: DGND -> ACOM
- C9 pad 2: DGND -> ACOM
- C90 pad 2: DGND -> ACOM
- C91 pad 2: DGND -> ACOM
- C92 pad 2: DGND -> ACOM
- C93 pad 2: DGND -> ACOM
- C94 pad 2: DGND -> ACOM
- C95 pad 2: DGND -> ACOM
- C96 pad 2: DGND -> ACOM
- C97 pad 2: DGND -> ACOM
- C98 pad 2: DGND -> ACOM
- C99 pad 2: DGND -> ACOM
- D2 pad 2: DGND -> ACOM
- D3 pad 2: DGND -> ACOM
- D4 pad 1: DGND -> ACOM
- FL1 pad 4: DGND -> ACOM
- H1 pad 1: DGND -> ACOM
- H10 pad 1: DGND -> ACOM
- H11 pad 1: DGND -> ACOM
- H12 pad 1: DGND -> ACOM
- H2 pad 1: DGND -> ACOM
- H3 pad 1: DGND -> ACOM
- H4 pad 1: DGND -> ACOM
- H5 pad 1: DGND -> ACOM
- H6 pad 1: DGND -> ACOM
- H7 pad 1: DGND -> ACOM
- H8 pad 1: DGND -> ACOM
- H9 pad 1: DGND -> ACOM
- J10 pad 2: DGND -> ACOM
- J11 pad 5: DGND -> ACOM
- J11 pad 6: DGND -> ACOM
- J12 pad 11: DGND -> ACOM
- J12 pad 6: DGND -> ACOM
- J13 pad 11: DGND -> ACOM
- J14 pad 4: DGND -> ACOM
- J14 pad 5: DGND -> ACOM
- J15 pad 11: DGND -> ACOM
- J15 pad 17: DGND -> ACOM
- J15 pad 2: DGND -> ACOM
- J15 pad 5: DGND -> ACOM
- J15 pad 8: DGND -> ACOM
- J15 pad SH: DGND -> ACOM
- J8 pad 6: DGND -> ACOM
- J9 pad 2: DGND -> ACOM
- JP1 pad 2: DGND -> ACOM
- JP2 pad 2: DGND -> ACOM
- JP3 pad 2: DGND -> ACOM
- JP4 pad 2: DGND -> ACOM
- JP5 pad 2: DGND -> ACOM
- L10 pad 2: DGND -> ACOM
- L9 pad 2: DGND -> ACOM
- LD1 pad 2: DGND -> ACOM
- LD11 pad 2: DGND -> ACOM
- LD12 pad 2: DGND -> ACOM
- LD2 pad 1: DGND -> ACOM
- LD2 pad 2: DGND -> ACOM
- LD2 pad 3: DGND -> ACOM
- LD3 pad 1: DGND -> ACOM
- LD3 pad 2: DGND -> ACOM
- LD3 pad 3: DGND -> ACOM
- LD4 pad 1: DGND -> ACOM
- LD4 pad 2: DGND -> ACOM
- LD4 pad 3: DGND -> ACOM
- LD5 pad 1: DGND -> ACOM
- LD5 pad 2: DGND -> ACOM
- LD5 pad 3: DGND -> ACOM
- LD6 pad 1: DGND -> ACOM
- LD6 pad 2: DGND -> ACOM
- LD6 pad 3: DGND -> ACOM
- LD7 pad 1: DGND -> ACOM
- LD7 pad 2: DGND -> ACOM
- LD7 pad 3: DGND -> ACOM
- LD8 pad 2: DGND -> ACOM
- LD9 pad 2: DGND -> ACOM
- Q11 pad 1: DGND -> ACOM
- Q12 pad 1: DGND -> ACOM
- Q13 pad 1: DGND -> ACOM
- Q2 pad 1: DGND -> ACOM
- Q4 pad 1: DGND -> ACOM
- Q7 pad 1: DGND -> ACOM
- Q9 pad 1: DGND -> ACOM
- R100 pad 2: DGND -> ACOM
- R107 pad 1: DGND -> ACOM
- R111 pad 2: DGND -> ACOM
- R112 pad 2: DGND -> ACOM
- R126 pad 2: DGND -> ACOM
- R127 pad 2: DGND -> ACOM
- R138 pad 2: DGND -> ACOM
- R139 pad 2: DGND -> ACOM
- R140 pad 2: DGND -> ACOM
- R141 pad 2: DGND -> ACOM
- R142 pad 2: DGND -> ACOM
- R15 pad 2: DGND -> ACOM
- R16 pad 2: DGND -> ACOM
- R26 pad 2: DGND -> ACOM
- R27 pad 2: DGND -> ACOM
- R28 pad 2: DGND -> ACOM
- R38 pad 2: DGND -> ACOM
- R39 pad 2: DGND -> ACOM
- R40 pad 2: DGND -> ACOM
- R43 pad 2: DGND -> ACOM
- R45 pad 2: DGND -> ACOM
- R47 pad 2: DGND -> ACOM
- R55 pad 2: DGND -> ACOM
- R56 pad 2: DGND -> ACOM
- R57 pad 2: DGND -> ACOM
- R62 pad 2: DGND -> ACOM
- R63 pad 4: Net-(C40-Pad1) -> Net-(C41-Pad1)
- R67 pad 2: DGND -> ACOM
- R68 pad 2: DGND -> ACOM
- R7 pad 2: DGND -> ACOM
- R75 pad 2: DGND -> ACOM
- R76 pad 2: DGND -> ACOM
- R77 pad 2: DGND -> ACOM
- R8 pad 2: DGND -> ACOM
- SW2 pad 3: DGND -> ACOM
- SW2 pad 4: DGND -> ACOM
- T1 pad 3: DGND -> ACOM
- U1 pad 8: DGND -> ACOM
- U10 pad 5: DGND -> ACOM
- U10 pad 8: DGND -> ACOM
- U10 pad 9: DGND -> ACOM
- U11 pad 1: DGND -> Net-(C117-Pad1)
- U11 pad 2: Net-(C40-Pad1) -> Net-(C41-Pad1)
- U11 pad 3: +5V -> Net-(C40-Pad1)
- U12 pad 5: DGND -> ACOM
- U13 pad 2: DGND -> ACOM
- U14 pad 49: DGND -> ACOM
- U15 pad 4: DGND -> ACOM
- U16 pad 10: DGND -> ACOM
- U16 pad 11: DGND -> ACOM
- U16 pad 14: DGND -> ACOM
- U16 pad 18: DGND -> ACOM
- U16 pad 2: DGND -> ACOM
- U16 pad 31: DGND -> ACOM
- U16 pad 4: DGND -> ACOM
- U16 pad 50: DGND -> ACOM
- U16 pad 61: DGND -> ACOM
- U16 pad 65: DGND -> ACOM
- U16 pad 7: DGND -> ACOM
- U17 pad 1.1: DGND -> ACOM
- U17 pad 1.19: DGND -> ACOM
- U17 pad 1.25: DGND -> ACOM
- U17 pad 1.30: DGND -> ACOM
- U17 pad 1.33: DGND -> ACOM
- U17 pad 1.43: DGND -> ACOM
- U17 pad 1.53: DGND -> ACOM
- U17 pad 1.54: DGND -> ACOM
- U17 pad 1.63: DGND -> ACOM
- U17 pad 1.64: DGND -> ACOM
- U17 pad 1.7: DGND -> ACOM
- U17 pad 1.73: DGND -> ACOM
- U17 pad 1.74: DGND -> ACOM
- U17 pad 1.83: DGND -> ACOM
- U17 pad 1.89: DGND -> ACOM
- U17 pad 2.10: VCCIO_B13 -> +3V3
- U17 pad 2.19: DGND -> ACOM
- U17 pad 2.29: DGND -> ACOM
- U17 pad 2.30: DGND -> ACOM
- U17 pad 2.39: DGND -> ACOM
- U17 pad 2.40: DGND -> ACOM
- U17 pad 2.49: DGND -> ACOM
- U17 pad 2.50: DGND -> ACOM
- U17 pad 2.59: DGND -> ACOM
- U17 pad 2.60: DGND -> ACOM
- U17 pad 2.69: DGND -> ACOM
- U17 pad 2.70: DGND -> ACOM
- U17 pad 2.79: DGND -> ACOM
- U17 pad 2.8: VCCIO_B13 -> +3V3
- U17 pad 2.80: DGND -> ACOM
- U17 pad 2.89: DGND -> ACOM
- U17 pad 3.11: DGND -> ACOM
- U17 pad 3.12: DGND -> ACOM
- U17 pad 3.17: DGND -> ACOM
- U17 pad 3.18: DGND -> ACOM
- U17 pad 3.23: DGND -> ACOM
- U17 pad 3.24: DGND -> ACOM
- U17 pad 3.29: DGND -> ACOM
- U17 pad 3.30: DGND -> ACOM
- U17 pad 3.35: DGND -> ACOM
- U17 pad 3.36: DGND -> ACOM
- U17 pad 3.45: DGND -> ACOM
- U17 pad 3.46: DGND -> ACOM
- U17 pad 3.5: DGND -> ACOM
- U17 pad 3.55: DGND -> ACOM
- U17 pad 3.6: DGND -> ACOM
- U17 pad SH1: DGND -> ACOM
- U17 pad SH2: DGND -> ACOM
- U17 pad SH3: DGND -> ACOM
- U18 pad 1: DGND -> ACOM
- U18 pad 14: DGND -> ACOM
- U18 pad 7: DGND -> ACOM
- U19 pad 2: DGND -> ACOM
- U2 pad 5: DGND -> ACOM
- U20 pad 11: DGND -> ACOM
- U20 pad 2: DGND -> ACOM
- U20 pad 25: DGND -> ACOM
- U21 pad 2: DGND -> ACOM
- U22 pad 2: DGND -> ACOM
- U23 pad 17: DGND -> Net-(U23-Pad17)
- U23 pad 2: DGND -> Net-(U23-Pad17)
- U24 pad 13: DGND -> ACOM
- U24 pad 14: DGND -> ACOM
- U24 pad 16: DGND -> ACOM
- U24 pad 17: DGND -> ACOM
- U24 pad 20: DGND -> ACOM
- U24 pad 26: DGND -> ACOM
- U24 pad 32: DGND -> ACOM
- U24 pad 34: DGND -> ACOM
- U24 pad 35: DGND -> ACOM
- U24 pad 40: DGND -> ACOM
- U24 pad 41: DGND -> ACOM
- U24 pad 42: DGND -> ACOM
- U24 pad 43: DGND -> ACOM
- U24 pad 48: DGND -> ACOM
- U24 pad 50: DGND -> ACOM
- U24 pad 51: DGND -> ACOM
- U24 pad 52: DGND -> ACOM
- U24 pad 53: DGND -> ACOM
- U24 pad 56: DGND -> ACOM
- U24 pad 60: DGND -> ACOM
- U24 pad 61: DGND -> ACOM
- U24 pad 62: DGND -> ACOM
- U24 pad 63: DGND -> ACOM
- U24 pad 64: DGND -> ACOM
- U24 pad 65: DGND -> ACOM
- U26 pad 22: DGND -> ACOM
- U26 pad 25: DGND -> ACOM
- U28 pad 22: DGND -> ACOM
- U28 pad 25: DGND -> ACOM
- U3 pad 2: DGND -> ACOM
- U30 pad 22: DGND -> ACOM
- U30 pad 25: DGND -> ACOM
- U32 pad 22: DGND -> ACOM
- U32 pad 25: DGND -> ACOM
- U34 pad 22: DGND -> ACOM
- U34 pad 25: DGND -> ACOM
- U4 pad 8: DGND -> ACOM
- U5 pad 5: DGND -> ACOM
- U6 pad 2: DGND -> ACOM
- U7 pad 1: DGND -> ACOM
- U8 pad 5: DGND -> ACOM
- U9 pad 2: DGND -> ACOM
- Y1 pad 2: DGND -> ACOM
Routing:
- net ACOM: track 0.00 -> 905.1 mm, vias 0 -> 659
- net DGND: track 904.2 -> 0.00 mm, vias 642 -> 0
- net 1V8_from_FPGA: track 50.1 -> 33.8 mm
- net +3.3VADC: track 40.3 -> 27.2 mm, vias 7 -> 3
- net +5V: track 23.1 -> 11.9 mm, vias 17 -> 13
- net Net-(J10-Pad1): track 14.8 -> 8.97 mm
- net MON_SCL: track 27.7 -> 22.2 mm
- net MON_SDA: track 28.1 -> 22.5 mm
- net Net-(C118-Pad1): track 0.00 -> 5.30 mm
- net Net-(R115-Pad2): track 4.44 -> 9.44 mm
- net ~PS_RESET: track 28.6 -> 24.6 mm
- net Net-(C117-Pad1): track 0.00 -> 3.43 mm
- net /Power Supply/Stage 3 Regulators/ADC 3V3 Monitor/Vin: track 6.22 -> 3.01 mm
- net VCCIO_B13: track 2.95 -> 0.00 mm, vias 3 -> 1
- net +3V3: track 156.2 -> 159.2 mm, vias 75 -> 77
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- added copper zone on B.Cu, net ACOM
- added copper zone on F.Cu, net ACOM
- added copper zone on In1.Cu, net ACOM
- added copper zone on F.Cu, net Net-(C41-Pad1)
- removed copper zone on F.Cu, net +3.3VADC
- removed copper zone on In2.Cu, net +3.3VADC
- removed copper zone on In2.Cu, net +5V
- removed copper zone on In2.Cu, net 3V3_LP
- removed copper zone on B.Cu, net DGND
- removed copper zone on F.Cu, net DGND
- removed copper zone on In1.Cu, net DGND
- removed copper zone on F.Cu, net Net-(C40-Pad1)
Other:
- board text removed: "PS Reset"
