File: v1.kicad_pcb (KiCad board)
At the start: 4 copper layers, 200 x 150 mm, 411 parts, among them J1 Powerpole G1377G2, J10 Conn_Coaxial, J11 USB_B_Micro, J12 Micro_SD_Card_Det, J13 ARJM11D7-502-AB-EW2, J14 USB_A, J15 HDMI_A, J16 Conn_Coaxial, J2 Barrel_Jack_Switch, J3 Conn_01x02, J4 Conn_01x02, J5 Conn_01x02, J6 Conn_01x02, J7 Conn_01x02, J8 Conn_01x06_Male, J9 Conn_Coaxial, M1 Logo_16mmx16mm, Q1 Si7141DP, Q10 Si7141DP, Q11 SI1539CDL-T1-GE3, Q12 SI1539CDL-T1-GE3, Q13 SI1539CDL-T1-GE3, Q2 SI1539CDL-T1-GE3, Q3 Si7141DP, Q4 SI1539CDL-T1-GE3, Q5 Si7141DP, Q6 Si7141DP, Q7 SI1539CDL-T1-GE3, Q8 Si7141DP, Q9 SI1539CDL-T1-GE3, SW1 SW_SPDT, SW2 Tactile_Switch_Generic, T1 PWB2010L, T2 Macom_ETC1-1-13, T3 PWB2010L, U1 171050601, U10 MAX9612, U11 ADM7154, U12 MAX9612, U13 TPS3701DDCR, U14 LCMXO2-640HC-4SG48C, U15 REF5025IDGK, U16 LTC2216, U17 TE0720, U18 JTAG-SMT3, U19 TPD2S017, U2 MAX9612, U20 TXS02612, U21 TPS2051B, U22 TPD2S017, U23 AD5689BCPZ, U24 TFP410PAP, U25 AD9744_LFCSP, U26 TLC59281RGER, U28 TLC59281RGER, U3 TPS3701DDCR, U30 TLC59281RGER, U32 TLC59281RGER, U34 TLC59281RGER, U4 171050601, U5 MAX9612, U6 TPS3701DDCR, U7 NCP1117-3.3_TO252, U8 MAX9612, U9 TPS3701DDCR, Y1 SIT5001AC-3E-33N0-80.000000X

Commit message: so much broken :(
Parts:
- moved J8 369.7 mm to (265.6, -11.4)
- moved LD2 369.7 mm to (277.3, -32.1)
- moved LD3 369.7 mm to (272.1, -32.1)
- moved LD4 369.7 mm to (267.1, -32.1)
- moved LD5 369.7 mm to (262.1, -32.1)
- moved LD6 369.7 mm to (257.1, -32.1)
- moved LD7 369.7 mm to (242.1, -32.1)
- moved LD8 369.7 mm to (247.1, -32.1)
- moved LD9 369.7 mm to (252.1, -32.1)
- moved R100 369.7 mm to (288.3, -11.1)
- moved R78 369.7 mm to (278.8, -26.1)
- moved R79 369.7 mm to (277.3, -26.1)
- moved R80 369.7 mm to (275.8, -26.1)
- moved R81 369.7 mm to (273.6, -26.1)
- moved R82 369.7 mm to (272.1, -26.1)
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Routing:
- net JTAG_TDO: track 80.2 -> 2.90 mm, vias 2 -> 1
- net JTAG_TCK: track 79.8 -> 2.90 mm, vias 2 -> 1
- net JTAG_TMS: track 82.4 -> 5.64 mm, vias 2 -> 1
- net /HDMI/R3: track 73.3 -> 1.41 mm
- net /HDMI/R2: track 71.7 -> 1.27 mm
- net /HDMI/R1: track 70.3 -> 1.37 mm
- net /HDMI/R0: track 68.7 -> 1.00 mm
- net JTAG_TDI: track 80.0 -> 13.5 mm, vias 2 -> 1
- net ~VDMA_Underflow: track 69.9 -> 3.50 mm, vias 2 -> 0
- net /HDMI/G2: track 64.1 -> 0.00 mm
- net /HDMI/G3: track 65.6 -> 1.71 mm
- net ~VDMA_Lock: track 65.8 -> 3.12 mm, vias 2 -> 0
- net /HDMI/G1: track 62.6 -> 1.44 mm
- net /HDMI/G0: track 61.2 -> 2.01 mm
- net /HDMI/B3: track 50.2 -> 1.55 mm
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Other:
- outline, holes or cut-outs redrawn
- board text added: "No coffee before soldering these ->"
- board text removed: "<- No coffee before soldering these"

Commit message: just about finished fiddling to add the RF DAC
Parts:
- removed REF**: Shield_Masach_MS570-10_52.7x30.7x6mm_TH, Shield_WUT:Shield_Masach_MS570-10_52.7x30.7x6mm_TH
- removed the U25 at (28.0, 17.0)
- added C123: 1u, Capacitor_SMD:C_0603_1608Metric, F.Cu at (84.8, 51.0)
- added C124: 100n, Capacitor_SMD:C_0603_1608Metric, F.Cu at (86.5, 51.0)
- added C125: 100n, Capacitor_SMD:C_0603_1608Metric, F.Cu at (81.8, 55.8)
- added C126: 100n, Capacitor_SMD:C_0402_1005Metric, F.Cu at (72.0, 39.8)
- added C127: 100n, Capacitor_SMD:C_0402_1005Metric, F.Cu at (76.0, 37.2)
- added C128: 1u, Capacitor_SMD:C_0603_1608Metric, F.Cu at (68.5, 37.5)
- added C129: 100n, Capacitor_SMD:C_0402_1005Metric, F.Cu at (72.0, 41.7)
- added C130: 100n, Capacitor_SMD:C_0402_1005Metric, F.Cu at (74.9, 39.8)
- added C131: 100n, Capacitor_SMD:C_0402_1005Metric, F.Cu at (74.9, 41.7)
- added C132: 1u, Capacitor_SMD:C_0603_1608Metric, F.Cu at (68.5, 40.0)
- added FB15: Ferrite_Bead_Small, Resistor_SMD:R_0603_1608Metric, F.Cu at (83.2, 58.8)
- added FB16: Ferrite_Bead_Small, Resistor_SMD:R_0603_1608Metric, F.Cu at (72.5, 37.5)
- added FB17: Ferrite_Bead_Small, Resistor_SMD:R_0603_1608Metric, F.Cu at (68.5, 42.5)
- added H13: Shield, Shield_WUT:Shield_Masach_MS570-10_52.7x30.7x6mm_TH, F.Cu at (77.8, 46.0)
- added R142: DNF, Resistor_SMD:R_0603_1608Metric, F.Cu at (85.2, 47.2)
- added R143: 2k, Resistor_SMD:R_0603_1608Metric, F.Cu at (88.0, 54.0)
- added R144: 10k, Resistor_SMD:R_0603_1608Metric, F.Cu at (87.8, 42.0)
- added R145: 10k, Resistor_SMD:R_0603_1608Metric, F.Cu at (89.8, 54.0)
- added R146: 33, Resistor_SMD:R_0603_1608Metric, F.Cu at (104.0, 84.5)
- added R147: 1k, Resistor_SMD:R_0402_1005Metric, F.Cu at (93.0, 42.8)
- added RN7: R_Pack08, Resistor_SMD:R_Array_Convex_8x0602, F.Cu at (97.5, 45.8)
- added RN8: R_Pack08, Resistor_SMD:R_Array_Convex_8x0602, F.Cu at (97.5, 51.8)
- added U30: AD9744_LFCSP, Package_CSP:LFCSP-32-1EP_5x5mm_P0.5mm_EP3.25x3.25mm, F.Cu at (90.5, 47.2)
- added U31: ADR280RT, Package_TO_SOT_SMD:SOT-23, F.Cu at (81.8, 53.0)
- J16: moved to B.Cu
- moved C90 395.6 mm to (331.2, 96.5)
- moved D4 395.6 mm to (331.2, 94.8)
- moved SW2 395.6 mm to (331.2, 99.8)
- moved C25 372.3 mm to (135.7, 165.7), turned to 90 degrees
- moved L3 358.5 mm to (122.2, 162.0), turned to 0 degrees
- moved D1 342.8 mm to (114.2, 155.1), turned to 90 degrees
- moved C26 335.8 mm to (110.8, 155.4), turned to 180 degrees
- moved R43 335.7 mm to (110.8, 157.9), turned to 180 degrees
- moved Q5 331.6 mm to (108.8, 162.1), turned to 180 degrees
- moved D2 319.1 mm to (102.5, 157.8), turned to 90 degrees
- moved FL1 312.7 mm to (99.3, 165.6), turned to 0 degrees
- moved SW1 286.0 mm to (86.0, 161.8), turned to 0 degrees
- moved J1 265.2 mm to (75.5, 165.6), turned to 90 degrees
- moved H5 242.7 mm to (17.8, 140.5), turned to 180 degrees
- moved C114 237.9 mm to (238.8, 94.8)
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- renumbered C98 to C100, C99 to C101, C100 to C102, C101 to C103, C102 to C104, C103 to C105, C104 to C106, C105 to C107, C106 to C108, C107 to C109, C108 to C110, C109 to C111, C110 to C112, C111 to C113, C112 to C114, C113 to C115, C114 to C116, C115 to C117, C116 to C118, C117 to C41, C118 to C42, C41 to C43, C42 to C44, C43 to C45, C44 to C46, C45 to C47, C46 to C48, C48 to C50, C49 to C51, C50 to C52, C51 to C53, C52 to C54, C53 to C55, C54 to C56, C55 to C57, C56 to C58, C57 to C59, C58 to C60, C59 to C61, C60 to C62, C61 to C63, C62 to C64, C63 to C65, C64 to C66, C65 to C67, C66 to C68, C67 to C69, C68 to C70, C69 to C71, C70 to C72, C71 to C73, C72 to C74, C73 to C75, C74 to C76, C75 to C77, C76 to C78, C77 to C79, C78 to C80, C79 to C81, C80 to C82, C81 to C83, C82 to C84, C83 to C85, C84 to C86, C85 to C87, C86 to C88, C87 to C89, C88 to C90, C89 to C91, C90 to C92, C91 to C93, C92 to C94, C93 to C95, C94 to C96, C95 to C97, C96 to C98, C97 to C99, R135 to R134, R136 to R135, R137 to R136, R138 to R137, R139 to R138, R140 to R139, R141 to R140, R142 to R141, U24 to U23, U26 to U24, U28 to U25, U30 to U26, U32 to U27, U34 to U28, U23 to U29
Connections:
- FB3 pad 1: +1V8 -> +3V3
- RN1 pad 10: ADC_D0 -> RF_ADC_D0
- RN1 pad 11: ADC_D1 -> RF_ADC_D1
- RN1 pad 12: ADC_D2 -> RF_ADC_D2
- RN1 pad 13: ADC_D3 -> RF_ADC_D3
- RN1 pad 14: ADC_D4 -> RF_ADC_D4
- RN1 pad 15: ADC_D5 -> RF_ADC_D5
- RN1 pad 16: ADC_D6 -> RF_ADC_D6
- RN1 pad 9: ADC_Clk -> ADC_Clk_N
- RN2 pad 10: ADC_D8 -> RF_ADC_D8
- RN2 pad 11: ADC_D9 -> RF_ADC_D9
- RN2 pad 12: ADC_D10 -> RF_ADC_D10
- RN2 pad 13: ADC_D11 -> RF_ADC_D11
- RN2 pad 14: ADC_D12 -> RF_ADC_D12
- RN2 pad 15: ADC_D13 -> RF_ADC_D13
- RN2 pad 16: ADC_D14 -> RF_ADC_D14
- RN2 pad 9: ADC_D7 -> RF_ADC_D7
- RN3 pad 5: ADC_D15 -> RF_ADC_D15
- RN3 pad 6: ADC_Overflow -> RF_ADC_Overflow
- RN3 pad 7: ADC_RAND -> RF_ADC_Random
- U17 pad 2.52: Net-(U17-Pad2.52) -> ADC_Clk_P
- U17 pad 2.54: Net-(U17-Pad2.54) -> ADC_Clk_N
- U17 pad 2.56: Net-(U17-Pad2.56) -> RF_ADC_D0
- U17 pad 2.58: Net-(U17-Pad2.58) -> RF_ADC_D1
- U17 pad 2.61: HDMI_R3 -> RF_DAC_D13
- U17 pad 2.62: Net-(U17-Pad2.62) -> RF_ADC_D2
- U17 pad 2.63: HDMI_R2 -> RF_DAC_D12
- U17 pad 2.64: Net-(U17-Pad2.64) -> RF_ADC_D3
- U17 pad 2.65: HDMI_R1 -> RF_DAC_D11
- U17 pad 2.66: Net-(U17-Pad2.66) -> RF_ADC_D4
- U17 pad 2.67: HDMI_R0 -> RF_DAC_D10
- U17 pad 2.68: Net-(U17-Pad2.68) -> RF_ADC_D5
- U17 pad 2.71: HDMI_G3 -> RF_DAC_D9
- U17 pad 2.72: Net-(U17-Pad2.72) -> RF_ADC_D6
- U17 pad 2.73: HDMI_G2 -> RF_DAC_D8
- U17 pad 2.74: Net-(U17-Pad2.74) -> RF_ADC_D7
- U17 pad 2.75: HDMI_G1 -> RF_DAC_D7
- U17 pad 2.76: Net-(U17-Pad2.76) -> RF_ADC_D8
- U17 pad 2.77: HDMI_G0 -> RF_DAC_D6
- U17 pad 2.78: Net-(U17-Pad2.78) -> RF_ADC_D9
- U17 pad 2.81: HDMI_B3 -> RF_DAC_D5
- U17 pad 2.82: Net-(U17-Pad2.82) -> RF_ADC_D10
- U17 pad 2.83: HDMI_B2 -> RF_DAC_D4
- U17 pad 2.84: Net-(U17-Pad2.84) -> RF_ADC_D11
- U17 pad 2.85: HDMI_CLK -> RF_DAC_D3
- U17 pad 2.86: Net-(U17-Pad2.86) -> RF_ADC_D12
- U17 pad 2.87: HDMI_B1 -> RF_DAC_D2
- U17 pad 2.88: ~VDMA_Underflow -> RF_ADC_D13
- U17 pad 2.90: ~VDMA_Lock -> RF_ADC_D14
- U17 pad 2.91: HDMI_B0 -> RF_DAC_D1
- U17 pad 2.93: HDMI_Active -> RF_DAC_D0
- U17 pad 2.95: HDMI_HSync -> RF_DAC_CLK_P
- U17 pad 2.97: HDMI_VSync -> RF_DAC_CLK_N
Routing:
- net ACOM: track 904.7 -> 922.9 mm, vias 646 -> 667
- net USB_OTG_VBUS: track 68.3 -> 52.7 mm
- net JTAG_TDI: track 13.5 -> 0.00 mm, vias 1 -> 0
- net USB_OTG_D-: track 79.7 -> 66.9 mm
- net USB_OTG_D+: track 78.2 -> 68.0 mm
- net Net-(RN8-Pad8): track 0.00 -> 9.67 mm
- net Net-(R120-Pad1): track 17.6 -> 8.34 mm, vias 2 -> 1
- net Net-(RN8-Pad7): track 0.00 -> 8.82 mm
- net /RF DAC/Clk_N: track 0.00 -> 8.70 mm
- net MON_SCL: track 22.2 -> 13.8 mm, vias 3 -> 2
- net Net-(RN8-Pad6): track 0.00 -> 7.97 mm
- net /RF DAC/Clk_P: track 0.00 -> 7.95 mm
- net Net-(C123-Pad1): track 0.00 -> 7.53 mm
- net Net-(R142-Pad2): track 0.00 -> 7.12 mm
- net Net-(R142-Pad1): track 0.00 -> 7.12 mm
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- added copper zone on In2.Cu, net ACOM
- removed copper zone on In2.Cu, net DGND

Commit message: board nearly back in sane state after adding RF DAC
Parts:
- removed C126: 100n, Capacitor_SMD:C_0402_1005Metric
- removed J1: Powerpole G1377G2, Connector_WUT:Powerpole_PP30-with-1377G2-PCB-pins-25A
- removed R100: 10k, Resistor_SMD:R_0603_1608Metric
- removed R27, R28, R36, R37, R39, R40, R53, R54, R56, R57, R73, R74, R76, R77: R, Resistor_SMD:R_0603_1608Metric
- removed R98, R99: 4k7, Resistor_SMD:R_0603_1608Metric
- added RN9: 5k1, Resistor_SMD:R_Array_Convex_8x0602, F.Cu at (223.5, 82.5)
- H13: footprint Shield_WUT:Shield_Masach_MS570-10_52.7x30.7x6mm_TH -> Shield_WUT:Shield_Masach_MS511-10_51.1x25.7x6.5mm_TH
- R24: value R -> 10k
- R25: value R -> 22k
- moved C30 432.8 mm to (141.8, 150.8), turned to 90 degrees
- moved R45 431.5 mm to (141.3, 174.2), turned to 0 degrees
- moved R49 431.3 mm to (141.3, 172.2), turned to 0 degrees
- moved C32 431.2 mm to (141.3, 170.2), turned to 0 degrees
- moved R47 430.2 mm to (140.8, 157.9), turned to 0 degrees
- moved C31 427.9 mm to (139.2, 149.8), turned to 180 degrees
- moved R52 427.7 mm to (139.2, 151.5), turned to 180 degrees
- moved U8 427.4 mm to (139.2, 154.5), turned to 0 degrees
- moved R44 424.0 mm to (137.6, 174.2), turned to 0 degrees
- moved U9 423.7 mm to (137.6, 170.2), turned to 0 degrees
- moved R46 423.7 mm to (137.6, 157.9), turned to 0 degrees
- moved R51 423.6 mm to (137.6, 167.2), turned to 180 degrees
- moved R42 416.5 mm to (133.8, 174.2), turned to 0 degrees
- moved J5 413.9 mm to (132.5, 155.2), turned to 0 degrees
- moved C34 411.0 mm to (141.3, 166.0), turned to 270 degrees
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Connections:
- net ADC_Clk renamed Net-(U17-Pad1.76)
- net ADC_D0 renamed Net-(U17-Pad1.72)
- net ADC_D1 renamed Net-(U17-Pad1.70)
- net ADC_D10 renamed Net-(U17-Pad1.48)
- net ADC_D11 renamed Net-(U17-Pad1.46)
- net ADC_D12 renamed Net-(U17-Pad1.44)
- net ADC_D13 renamed Net-(U17-Pad1.42)
- net ADC_D14 renamed Net-(U17-Pad1.38)
- net ADC_D15 renamed Net-(U17-Pad1.36)
- net ADC_D2 renamed Net-(U17-Pad1.68)
- net ADC_D3 renamed Net-(U17-Pad1.66)
- net ADC_D4 renamed Net-(U17-Pad1.62)
- net ADC_D5 renamed Net-(U17-Pad1.60)
- net ADC_D6 renamed Net-(U17-Pad1.58)
- net ADC_D7 renamed Net-(U17-Pad1.56)
- net ADC_D8 renamed Net-(U17-Pad1.52)
- net ADC_D9 renamed Net-(U17-Pad1.50)
- net ADC_DITH renamed /RF ADC/ADC_Dither
- net ADC_RAND renamed Net-(U17-Pad1.32)
- Q12 pad 2: ADC_Overflow -> RF_ADC_Overflow
- R120 pad 1: Net-(R120-Pad1) -> RF_ADC_Dither
- R146 pad 1: ADC_Clk_P -> RF_ADC_Clk_P
- R24 pad 2: Net-(R24-Pad2) -> /Power Supply/Stage 3 Regulators/ADC 3V3 Monitor/A0
- R25 pad 1: 3V3_LP -> /Power Supply/Stage 3 Regulators/ADC 3V3 Monitor/A0
- R25 pad 2: Net-(R25-Pad2) -> ACOM
- RN1 pad 9: ADC_Clk_N -> RF_ADC_Clk_N
- U10 pad 8: ACOM -> 3V3_LP
- U10 pad 9: ACOM -> 3V3_LP
- U12 pad 8: Net-(R74-Pad2) -> ACOM
- U12 pad 9: Net-(R73-Pad2) -> /Power Supply/Stage 3 Regulators/ADC 3V3 Monitor/A0
- U17 pad 1.34: ADC_Overflow -> Net-(U17-Pad1.34)
- U17 pad 1.78: Net-(R120-Pad1) -> Net-(U17-Pad1.78)
- U17 pad 2.47: Net-(U17-Pad2.47) -> RF_ADC_Dither
- U17 pad 2.51: Net-(U17-Pad2.51) -> RF_ADC_Clk_P
- U17 pad 2.52: ADC_Clk_P -> RF_DAC_D13
- U17 pad 2.53: Net-(U17-Pad2.53) -> RF_ADC_Clk_N
- U17 pad 2.54: ADC_Clk_N -> RF_DAC_D12
- U17 pad 2.55: Net-(U17-Pad2.55) -> RF_ADC_D0
- U17 pad 2.56: RF_ADC_D0 -> RF_DAC_D11
- U17 pad 2.57: Net-(U17-Pad2.57) -> RF_ADC_D1
- U17 pad 2.58: RF_ADC_D1 -> RF_DAC_D10
- U17 pad 2.61: RF_DAC_D13 -> RF_ADC_D2
- U17 pad 2.62: RF_ADC_D2 -> RF_DAC_D9
- U17 pad 2.63: RF_DAC_D12 -> RF_ADC_D3
- U17 pad 2.64: RF_ADC_D3 -> RF_DAC_D8
- U17 pad 2.65: RF_DAC_D11 -> RF_ADC_D4
- U17 pad 2.66: RF_ADC_D4 -> RF_DAC_D7
- U17 pad 2.67: RF_DAC_D10 -> RF_ADC_D5
- U17 pad 2.68: RF_ADC_D5 -> RF_DAC_D6
- U17 pad 2.71: RF_DAC_D9 -> RF_ADC_D6
- U17 pad 2.72: RF_ADC_D6 -> RF_DAC_D5
- U17 pad 2.73: RF_DAC_D8 -> RF_ADC_D7
- U17 pad 2.74: RF_ADC_D7 -> RF_DAC_D4
- U17 pad 2.75: RF_DAC_D7 -> RF_ADC_D8
- U17 pad 2.76: RF_ADC_D8 -> RF_DAC_D3
- U17 pad 2.77: RF_DAC_D6 -> RF_ADC_D9
- U17 pad 2.78: RF_ADC_D9 -> RF_DAC_D2
- U17 pad 2.81: RF_DAC_D5 -> RF_ADC_D10
- U17 pad 2.82: RF_ADC_D10 -> RF_DAC_D1
- U17 pad 2.83: RF_DAC_D4 -> RF_ADC_D11
- U17 pad 2.84: RF_ADC_D11 -> RF_DAC_D0
- U17 pad 2.85: RF_DAC_D3 -> RF_ADC_D12
- U17 pad 2.86: RF_ADC_D12 -> RF_DAC_CLK_P
- U17 pad 2.87: RF_DAC_D2 -> RF_ADC_D13
- U17 pad 2.88: RF_ADC_D13 -> RF_DAC_CLK_N
- U17 pad 2.90: RF_ADC_D14 -> Net-(U17-Pad2.90)
- U17 pad 2.91: RF_DAC_D1 -> RF_ADC_D14
- U17 pad 2.93: RF_DAC_D0 -> RF_ADC_D15
- U17 pad 2.95: RF_DAC_CLK_P -> RF_ADC_Overflow
- U17 pad 2.97: RF_DAC_CLK_N -> RF_ADC_Random
- U2 pad 8: Net-(R25-Pad2) -> ACOM
- U2 pad 9: Net-(R24-Pad2) -> 3V3_LP
- U5 pad 8: Net-(R37-Pad2) -> 3V3_LP
- U5 pad 9: Net-(R36-Pad2) -> ACOM
- U8 pad 8: Net-(R54-Pad2) -> ACOM
- U8 pad 9: Net-(R53-Pad2) -> ACOM
Routing:
- net MON_SDA: track 15.5 -> 178.4 mm, vias 2 -> 7
- net MON_SCL: track 13.8 -> 176.1 mm, vias 2 -> 5
- net FPGA_PWR_GOOD: track 8.54 -> 59.6 mm, vias 0 -> 2
- net RF_DAC_D5: track 0.00 -> 49.6 mm, vias 0 -> 2
- net RF_DAC_D0: track 0.00 -> 49.6 mm, vias 0 -> 2
- net RF_DAC_D3: track 0.00 -> 49.5 mm, vias 0 -> 2
- net RF_DAC_D11: track 0.00 -> 49.1 mm, vias 0 -> 2
- net RF_DAC_D6: track 0.00 -> 48.9 mm, vias 0 -> 2
- net RF_DAC_CLK_N: track 0.00 -> 48.8 mm, vias 0 -> 2
- net RF_DAC_D8: track 0.00 -> 48.7 mm, vias 0 -> 2
- net RF_DAC_D13: track 0.00 -> 48.6 mm, vias 0 -> 2
- net RF_DAC_D4: track 0.00 -> 47.3 mm, vias 0 -> 2
- net RF_DAC_D2: track 0.00 -> 47.3 mm, vias 0 -> 2
- net RF_DAC_D7: track 0.00 -> 46.9 mm, vias 0 -> 2
- net RF_DAC_D12: track 0.00 -> 46.9 mm, vias 0 -> 2
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- added copper zone on F.Cu, net +3.3VADC
- added copper zone on In2.Cu, net +5V
- added copper zone on F.Cu, net 3V3_LP
- added copper zone on In2.Cu, net 3V3_LP
Other:
- outline, holes or cut-outs redrawn
- board text added: "EN"
- board text added: "FPGA PWR"
- board text added: "Guard dog stops EMI getting into the cans"
- board text added: "MODE"
- board text added: "OTG"

Commit message: made it to the painful stage - 40 traces to go (plus bells and whistles need adding)
Parts:
- removed U29: AD5689BCPZ, Package_CSP:LFCSP-16-1EP_3x3mm_P0.5mm_EP1.854x1.854mm
- added C126: DNF, Capacitor_SMD:C_0603_1608Metric, F.Cu at (199.2, 91.5)
- added RN10: 33, Resistor_SMD:R_Array_Convex_8x0602, F.Cu at (167.0, 81.2)
- moved RN5 88.8 mm to (167.0, 71.2), turned to 0 degrees
- moved RN6 88.8 mm to (167.0, 76.2), turned to 0 degrees
- moved C114 58.8 mm to (180.0, 92.8)
- moved LD14 58.8 mm to (180.0, 106.8)
- moved R137 58.8 mm to (180.0, 91.0)
- moved U24 58.8 mm to (180.0, 96.2)
- moved C118 57.2 mm to (238.0, 92.8)
- moved LD18 57.2 mm to (238.0, 106.8)
- moved R141 57.2 mm to (238.0, 91.0)
- moved U28 57.2 mm to (238.0, 96.2)
- moved C115 29.8 mm to (194.5, 92.8)
- moved LD15 29.8 mm to (194.5, 106.8)
- moved R138 29.8 mm to (194.5, 91.0)
- moved U25 29.8 mm to (194.5, 96.2)
- moved C117 28.2 mm to (223.5, 92.8)
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Connections:
- RN5 pad 1: HDMI_B3 -> HDMI_R4
- RN5 pad 10: /HDMI/HSync -> /HDMI/G4
- RN5 pad 11: /HDMI/Active -> /HDMI/G5
- RN5 pad 12: /HDMI/B0 -> /HDMI/R0
- RN5 pad 13: /HDMI/B1 -> /HDMI/R1
- RN5 pad 14: /HDMI/Clk -> /HDMI/R2
- RN5 pad 15: /HDMI/B2 -> /HDMI/R3
- RN5 pad 16: /HDMI/B3 -> /HDMI/R4
- RN5 pad 2: HDMI_B2 -> HDMI_R3
- RN5 pad 3: HDMI_CLK -> HDMI_R2
- RN5 pad 4: HDMI_B1 -> HDMI_R1
- RN5 pad 5: HDMI_B0 -> HDMI_R0
- RN5 pad 6: HDMI_Active -> HDMI_G5
- RN5 pad 7: HDMI_HSync -> HDMI_G4
- RN5 pad 8: HDMI_VSync -> HDMI_G3
- RN5 pad 9: /HDMI/VSync -> /HDMI/G3
- RN6 pad 1: HDMI_R3 -> HDMI_G2
- RN6 pad 10: /HDMI/G1 -> /HDMI/B2
- RN6 pad 11: /HDMI/G2 -> /HDMI/Clk
- RN6 pad 12: /HDMI/G3 -> /HDMI/B3
- RN6 pad 13: /HDMI/R0 -> /HDMI/B4
- RN6 pad 14: /HDMI/R1 -> /HDMI/G0
- RN6 pad 15: /HDMI/R2 -> /HDMI/G1
- RN6 pad 16: /HDMI/R3 -> /HDMI/G2
- RN6 pad 2: HDMI_R2 -> HDMI_G1
- RN6 pad 3: HDMI_R1 -> HDMI_G0
- RN6 pad 4: HDMI_R0 -> HDMI_B4
- RN6 pad 5: HDMI_G3 -> HDMI_B3
- RN6 pad 6: HDMI_G2 -> HDMI_Clk
- RN6 pad 7: HDMI_G1 -> HDMI_B2
- RN6 pad 8: HDMI_G0 -> HDMI_B1
- RN6 pad 9: /HDMI/G0 -> /HDMI/B1
- U17 pad 1.36: Net-(U17-Pad1.36) -> HDMI_VSync
- U17 pad 1.38: Net-(U17-Pad1.38) -> HDMI_HSync
- U17 pad 1.42: Net-(U17-Pad1.42) -> HDMI_Active
- U17 pad 1.44: Net-(U17-Pad1.44) -> HDMI_B0
- U17 pad 1.46: Net-(U17-Pad1.46) -> HDMI_B1
- U17 pad 1.48: Net-(U17-Pad1.48) -> HDMI_B2
- U17 pad 1.50: Net-(U17-Pad1.50) -> HDMI_Clk
- U17 pad 1.52: Net-(U17-Pad1.52) -> HDMI_B3
- U17 pad 1.56: Net-(U17-Pad1.56) -> HDMI_B4
- U17 pad 1.58: Net-(U17-Pad1.58) -> HDMI_G0
- U17 pad 1.60: Net-(U17-Pad1.60) -> HDMI_G1
- U17 pad 1.62: Net-(U17-Pad1.62) -> HDMI_G2
- U17 pad 1.66: Net-(U17-Pad1.66) -> HDMI_G3
- U17 pad 1.68: Net-(U17-Pad1.68) -> HDMI_G4
- U17 pad 1.70: Net-(U17-Pad1.70) -> HDMI_G5
- U17 pad 1.72: Net-(U17-Pad1.72) -> HDMI_R0
- U17 pad 1.76: Net-(U17-Pad1.76) -> HDMI_R1
- U17 pad 1.78: Net-(U17-Pad1.78) -> HDMI_R2
- U17 pad 1.82: Net-(U17-Pad1.82) -> HDMI_R3
- U17 pad 1.84: Net-(U17-Pad1.84) -> HDMI_R4
- U17 pad 1.85: Net-(U17-Pad1.85) -> ~VDMA_Lock
- U17 pad 1.87: Net-(U17-Pad1.87) -> ~VDMA_Underflow
- U23 pad 36: /HDMI/R3 -> /HDMI/R4
- U23 pad 37: /HDMI/R2 -> /HDMI/R3
- U23 pad 38: /HDMI/R1 -> /HDMI/R2
- U23 pad 39: /HDMI/R0 -> /HDMI/R1
- U23 pad 40: ACOM -> /HDMI/R0
- U23 pad 44: /HDMI/G3 -> /HDMI/G5
- U23 pad 45: /HDMI/G2 -> /HDMI/G4
- U23 pad 46: /HDMI/G1 -> /HDMI/G3
- U23 pad 47: /HDMI/G0 -> /HDMI/G2
- U23 pad 50: ACOM -> /HDMI/G1
- U23 pad 51: ACOM -> /HDMI/G0
- U23 pad 54: /HDMI/B3 -> /HDMI/B4
- U23 pad 55: /HDMI/B2 -> /HDMI/B3
- U23 pad 58: /HDMI/B1 -> /HDMI/B2
- U23 pad 59: /HDMI/B0 -> /HDMI/B1
- U23 pad 60: ACOM -> /HDMI/B0
Routing:
- net +5V: track 15.3 -> 139.2 mm, vias 15 -> 17
- net JTAG_TMS: track 0.00 -> 115.9 mm, vias 0 -> 2
- net JTAG_TDI: track 0.00 -> 113.8 mm, vias 0 -> 2
- net JTAG_TCK: track 0.00 -> 112.0 mm, vias 0 -> 2
- net JTAG_TDO: track 0.00 -> 108.8 mm, vias 0 -> 2
- net S2_PWR_ENABLE: track 45.6 -> 123.6 mm, vias 2 -> 3
- net LED_LAT: track 0.00 -> 73.6 mm, vias 0 -> 5
- net UART_DEBUG_TO_FPGA: track 0.00 -> 66.0 mm, vias 0 -> 2
- net LED_BLANK: track 0.00 -> 65.5 mm, vias 0 -> 5
- net LED_SCLK: track 0.00 -> 64.7 mm, vias 0 -> 5
- net UART_DEBUG_FROM_FPGA: track 0.00 -> 54.7 mm
- net /HDMI/VSync: track 5.59 -> 55.4 mm, vias 0 -> 2
- net /HDMI/HSync: track 5.38 -> 53.5 mm, vias 0 -> 2
- net /HDMI/Active: track 4.96 -> 51.8 mm, vias 0 -> 2
- net ~VDMA_Lock: track 0.00 -> 40.8 mm, vias 0 -> 2
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Other:
- board text added: "JTAG MODE"
- board text added: "NOSEQ"
